File: kicad/Row_A.sch (KiCad schematic (older format))
At the start: 10 parts, among them U01 APA102, U02 APA102, U03 APA102, U04 APA102, U05 APA102, U06 APA102, U07 APA102, U08 APA102

Commit message: UlTiM8x8 board layout complete, Gerbers ready for fab
Parts:
- C1: value 100n -> 100nF
- C2: value 47u,8V -> 47uF 20V
- renumbered U01 to U1, U02 to U2, U03 to U3, U04 to U4, U05 to U5, U06 to U6, U07 to U7, U08 to U8
Changed lines of the file:
@@
 P 1800 2600
 F 0 "C1" H 1825 2700 40  0000 L CNB
-F 1 "100n" H 1825 2500 40  0000 L CNN
+F 1 "100nF" H 1825 2500 40  0000 L CNN
 F 2 "ultim8x8_libs:c_0805" H 1800 2600 50  0001 C CNN
 F 3 "" H 1800 2600 60  0001 C CNN
@@
 P 1250 6750
 F 0 "C2" H 1375 6725 40  0000 L CNB
-F 1 "47u,8V" H 1375 6625 40  0000 L CNN
+F 1 "47uF 20V" H 1375 6625 40  0000 L CNN
 F 2 "ultim8x8_libs:c_2917" H 1250 6700 50  0001 C CNN
 F 3 "" H 1250 6750 60  0001 C CNN
@@
 GND
 $Comp
-L APA102 U01
+L APA102 U1
 U 1 1 56C2E1C1
 P 1700 1600
-F 0 "U01" H 1700 1900 40  0000 C CNB
+F 0 "U1" H 1700 1900 40  0000 C CNB
 F 1 "APA102" H 1700 1275 40  0000 C CNN
 F 2 "ultim8x8_libs:APA102" H 1600 2000 60  0001 C CNN
@@
 5V
 $Comp
-L APA102 U02
+L APA102 U2
 U 1 1 56C2E1EC
 P 2900 1600
-F 0 "U02" H 2900 1900 40  0000 C CNB
+F 0 "U2" H 2900 1900 40  0000 C CNB
 F 1 "APA102" H 2900 1275 40  0000 C CNN
 F 2 "ultim8x8_libs:APA102" H 2800 2000 60  0001 C CNN
@@
 $EndComp
 $Comp
-L APA102 U03
+L APA102 U3
 U 1 1 56C2E1F4
 P 4100 1600
-F 0 "U03" H 4100 1900 40  0000 C CNB
+F 0 "U3" H 4100 1900 40  0000 C CNB
 F 1 "APA102" H 4100 1275 40  0000 C CNN
 F 2 "ultim8x8_libs:APA102" H 4000 2000 60  0001 C CNN
@@
 $EndComp
 $Comp
-L APA102 U04
+L APA102 U4
 U 1 1 56C2E1FC
 P 5300 1600
-F 0 "U04" H 5300 1900 40  0000 C CNB
+F 0 "U4" H 5300 1900 40  0000 C CNB
 F 1 "APA102" H 5300 1275 40  0000 C CNN
 F 2 "ultim8x8_libs:APA102" H 5200 2000 60  0001 C CNN
@@
 $EndComp
 $Comp
-L APA102 U05
+L APA102 U5
 U 1 1 56C2E204
 P 6500 1600
-F 0 "U05" H 6500 1900 40  0000 C CNB
+F 0 "U5" H 6500 1900 40  0000 C CNB
 F 1 "APA102" H 6500 1275 40  0000 C CNN
 F 2 "ultim8x8_libs:APA102" H 6400 2000 60  0001 C CNN
@@
 $EndComp
 $Comp
-L APA102 U06
+L APA102 U6
 U 1 1 56C2E20C
 P 7700 1600
-F 0 "U06" H 7700 1900 40  0000 C CNB
+F 0 "U6" H 7700 1900 40  0000 C CNB
 F 1 "APA102" H 7700 1275 40  0000 C CNN
 F 2 "ultim8x8_libs:APA102" H 7600 2000 60  0001 C CNN
@@
 $EndComp
 $Comp
-L APA102 U07
+L APA102 U7
 U 1 1 56C2E214
 P 8900 1600
-F 0 "U07" H 8900 1900 40  0000 C CNB
+F 0 "U7" H 8900 1900 40  0000 C CNB
 F 1 "APA102" H 8900 1275 40  0000 C CNN
 F 2 "ultim8x8_libs:APA102" H 8800 2000 60  0001 C CNN
@@
 $EndComp
 $Comp
-L APA102 U08
+L APA102 U8
 U 1 1 56C2E21C
 P 10100 1600
-F 0 "U08" H 10100 1900 40  0000 C CNB
+F 0 "U8" H 10100 1900 40  0000 C CNB
 F 1 "APA102" H 10100 1275 40  0000 C CNN
 F 2 "ultim8x8_libs:APA102" H 10000 2000 60  0001 C CNN

Commit message: revised layout, final. Gerbers ready for fab
Parts:
- U05: renamed from U5; footprint ultim8x8_libs:APA102 -> ultim8x8_libs:APA102_U05
- U06: renamed from U6; footprint ultim8x8_libs:APA102 -> ultim8x8_libs:APA102_U06
- renumbered U1 to U01, U2 to U02, U3 to U03, U4 to U04, U7 to U07, U8 to U08
Changed lines of the file:
@@
 GND
 $Comp
-L APA102 U1
+L APA102 U01
 U 1 1 56C2E1C1
 P 1700 1600
-F 0 "U1" H 1700 1900 40  0000 C CNB
+F 0 "U01" H 1700 1900 40  0000 C CNB
 F 1 "APA102" H 1700 1275 40  0000 C CNN
 F 2 "ultim8x8_libs:APA102" H 1600 2000 60  0001 C CNN
@@
 5V
 $Comp
-L APA102 U2
+L APA102 U02
 U 1 1 56C2E1EC
 P 2900 1600
-F 0 "U2" H 2900 1900 40  0000 C CNB
+F 0 "U02" H 2900 1900 40  0000 C CNB
 F 1 "APA102" H 2900 1275 40  0000 C CNN
 F 2 "ultim8x8_libs:APA102" H 2800 2000 60  0001 C CNN
@@
 $EndComp
 $Comp
-L APA102 U3
+L APA102 U03
 U 1 1 56C2E1F4
 P 4100 1600
-F 0 "U3" H 4100 1900 40  0000 C CNB
+F 0 "U03" H 4100 1900 40  0000 C CNB
 F 1 "APA102" H 4100 1275 40  0000 C CNN
 F 2 "ultim8x8_libs:APA102" H 4000 2000 60  0001 C CNN
@@
 $EndComp
 $Comp
-L APA102 U4
+L APA102 U04
 U 1 1 56C2E1FC
 P 5300 1600
-F 0 "U4" H 5300 1900 40  0000 C CNB
+F 0 "U04" H 5300 1900 40  0000 C CNB
 F 1 "APA102" H 5300 1275 40  0000 C CNN
 F 2 "ultim8x8_libs:APA102" H 5200 2000 60  0001 C CNN
@@
 $EndComp
 $Comp
-L APA102 U5
+L APA102 U05
 U 1 1 56C2E204
 P 6500 1600
-F 0 "U5" H 6500 1900 40  0000 C CNB
+F 0 "U05" H 6500 1900 40  0000 C CNB
 F 1 "APA102" H 6500 1275 40  0000 C CNN
-F 2 "ultim8x8_libs:APA102" H 6400 2000 60  0001 C CNN
+F 2 "ultim8x8_libs:APA102_U05" H 6400 2000 60  0001 C CNN
 F 3 "" H 6500 1600 60  0001 C CNN
 F 4 "mfr_pn" H 6500 1600 60  0001 C CNN "manf#"
@@
 $EndComp
 $Comp
-L APA102 U6
+L APA102 U06
 U 1 1 56C2E20C
 P 7700 1600
-F 0 "U6" H 7700 1900 40  0000 C CNB
+F 0 "U06" H 7700 1900 40  0000 C CNB
 F 1 "APA102" H 7700 1275 40  0000 C CNN
-F 2 "ultim8x8_libs:APA102" H 7600 2000 60  0001 C CNN
+F 2 "ultim8x8_libs:APA102_U06" H 7600 2000 60  0001 C CNN
 F 3 "" H 7700 1600 60  0001 C CNN
 F 4 "mfr_pn" H 7700 1600 60  0001 C CNN "manf#"
@@
 $EndComp
 $Comp
-L APA102 U7
+L APA102 U07
 U 1 1 56C2E214
 P 8900 1600
-F 0 "U7" H 8900 1900 40  0000 C CNB
+F 0 "U07" H 8900 1900 40  0000 C CNB
 F 1 "APA102" H 8900 1275 40  0000 C CNN
 F 2 "ultim8x8_libs:APA102" H 8800 2000 60  0001 C CNN
@@
 $EndComp
 $Comp
-L APA102 U8
+L APA102 U08
 U 1 1 56C2E21C
 P 10100 1600
-F 0 "U8" H 10100 1900 40  0000 C CNB
+F 0 "U08" H 10100 1900 40  0000 C CNB
 F 1 "APA102" H 10100 1275 40  0000 C CNN
 F 2 "ultim8x8_libs:APA102" H 10000 2000 60  0001 C CNN
