File: kicad/Row_B.sch (KiCad schematic (older format))
At the start: 8 parts, among them U09 APA102, U10 APA102, U11 APA102, U12 APA102, U13 APA102, U14 APA102, U15 APA102, U16 APA102

Commit message: UlTiM8x8 board layout complete, Gerbers ready for fab
Parts:
- renumbered U09 to U9
Changed lines of the file:
@@
 GND
 $Comp
-L APA102 U09
+L APA102 U9
 U 1 1 56C2B784
 P 1700 1600
-F 0 "U09" H 1700 1900 40  0000 C CNB
+F 0 "U9" H 1700 1900 40  0000 C CNB
 F 1 "APA102" H 1700 1275 40  0000 C CNN
 F 2 "ultim8x8_libs:APA102" H 1600 2000 60  0001 C CNN

Commit message: revised layout, final. Gerbers ready for fab
Parts:
- U11: footprint ultim8x8_libs:APA102 -> ultim8x8_libs:APA102_U11
- U12: footprint ultim8x8_libs:APA102 -> ultim8x8_libs:APA102_U12
- renumbered U9 to U09
Changed lines of the file:
@@
 GND
 $Comp
-L APA102 U9
+L APA102 U09
 U 1 1 56C2B784
 P 1700 1600
-F 0 "U9" H 1700 1900 40  0000 C CNB
+F 0 "U09" H 1700 1900 40  0000 C CNB
 F 1 "APA102" H 1700 1275 40  0000 C CNN
 F 2 "ultim8x8_libs:APA102" H 1600 2000 60  0001 C CNN
@@
 F 0 "U11" H 4100 1900 40  0000 C CNB
 F 1 "APA102" H 4100 1275 40  0000 C CNN
-F 2 "ultim8x8_libs:APA102" H 4000 2000 60  0001 C CNN
+F 2 "ultim8x8_libs:APA102_U11" H 4000 2000 60  0001 C CNN
 F 3 "" H 4100 1600 60  0001 C CNN
 F 4 "mfr_pn" H 4100 1600 60  0001 C CNN "manf#"
@@
 F 0 "U12" H 5300 1900 40  0000 C CNB
 F 1 "APA102" H 5300 1275 40  0000 C CNN
-F 2 "ultim8x8_libs:APA102" H 5200 2000 60  0001 C CNN
+F 2 "ultim8x8_libs:APA102_U12" H 5200 2000 60  0001 C CNN
 F 3 "" H 5300 1600 60  0001 C CNN
 F 4 "mfr_pn" H 5300 1600 60  0001 C CNN "manf#"
