File: kicad/Row_C.sch (KiCad schematic (older format))
At the start: 8 parts, among them U17 APA102, U18 APA102, U19 APA102, U20 APA102, U21 APA102, U22 APA102, U23 APA102, U24 APA102

Commit message: revised layout, final. Gerbers ready for fab
Parts:
- U19: footprint ultim8x8_libs:APA102 -> ultim8x8_libs:APA102_U19
Changed lines of the file:
@@
 F 0 "U19" H 4100 1900 40  0000 C CNB
 F 1 "APA102" H 4100 1275 40  0000 C CNN
-F 2 "ultim8x8_libs:APA102" H 4000 2000 60  0001 C CNN
+F 2 "ultim8x8_libs:APA102_U19" H 4000 2000 60  0001 C CNN
 F 3 "" H 4100 1600 60  0001 C CNN
 F 4 "mfr_pn" H 4100 1600 60  0001 C CNN "manf#"
