File: kicad/Row_E.sch (KiCad schematic (older format))
At the start: 8 parts, among them U33 APA102, U34 APA102, U35 APA102, U36 APA102, U37 APA102, U38 APA102, U39 APA102, U40 APA102

Commit message: revised layout, final. Gerbers ready for fab
Parts:
- U38: footprint ultim8x8_libs:APA102 -> ultim8x8_libs:APA102_U38
Changed lines of the file:
@@
 F 0 "U38" H 7700 1900 40  0000 C CNB
 F 1 "APA102" H 7700 1275 40  0000 C CNN
-F 2 "ultim8x8_libs:APA102" H 7600 2000 60  0001 C CNN
+F 2 "ultim8x8_libs:APA102_U38" H 7600 2000 60  0001 C CNN
 F 3 "" H 7700 1600 60  0001 C CNN
 F 4 "mfr_pn" H 7700 1600 60  0001 C CNN "manf#"
