File: kicad/Row_F.sch (KiCad schematic (older format))
At the start: 8 parts, among them U41 APA102, U42 APA102, U43 APA102, U44 APA102, U45 APA102, U46 APA102, U47 APA102, U48 APA102

Commit message: revised layout, final. Gerbers ready for fab
Parts:
- U43: footprint ultim8x8_libs:APA102 -> ultim8x8_libs:APA102_U43
Changed lines of the file:
@@
 F 0 "U43" H 4100 1900 40  0000 C CNB
 F 1 "APA102" H 4100 1275 40  0000 C CNN
-F 2 "ultim8x8_libs:APA102" H 4000 2000 60  0001 C CNN
+F 2 "ultim8x8_libs:APA102_U43" H 4000 2000 60  0001 C CNN
 F 3 "" H 4100 1600 60  0001 C CNN
 F 4 "mfr_pn" H 4100 1600 60  0001 C CNN "manf#"
