File: kicad/Row_G.sch (KiCad schematic (older format))
At the start: 8 parts, among them U49 APA102, U50 APA102, U51 APA102, U52 APA102, U53 APA102, U54 APA102, U55 APA102, U56 APA102

Commit message: revised layout, final. Gerbers ready for fab
Parts:
- U53: footprint ultim8x8_libs:APA102 -> ultim8x8_libs:APA102_U53
- U54: footprint ultim8x8_libs:APA102 -> ultim8x8_libs:APA102_U54
Changed lines of the file:
@@
 F 0 "U53" H 6500 1900 40  0000 C CNB
 F 1 "APA102" H 6500 1275 40  0000 C CNN
-F 2 "ultim8x8_libs:APA102" H 6400 2000 60  0001 C CNN
+F 2 "ultim8x8_libs:APA102_U53" H 6400 2000 60  0001 C CNN
 F 3 "" H 6500 1600 60  0001 C CNN
 F 4 "mfr_pn" H 6500 1600 60  0001 C CNN "manf#"
@@
 F 0 "U54" H 7700 1900 40  0000 C CNB
 F 1 "APA102" H 7700 1275 40  0000 C CNN
-F 2 "ultim8x8_libs:APA102" H 7600 2000 60  0001 C CNN
+F 2 "ultim8x8_libs:APA102_U54" H 7600 2000 60  0001 C CNN
 F 3 "" H 7700 1600 60  0001 C CNN
 F 4 "mfr_pn" H 7700 1600 60  0001 C CNN "manf#"
