File: kicad/Row_H.sch (KiCad schematic (older format))
At the start: 10 parts, among them U57 APA102, U58 APA102, U59 APA102, U60 APA102, U61 APA102, U62 APA102, U63 APA102, U64 APA102

Commit message: UlTiM8x8 board layout complete, Gerbers ready for fab
Parts:
- C3: value 100n -> 100nF
- C4: value 47u,8V -> 47uF 20V
Changed lines of the file:
@@
 P 1800 2600
 F 0 "C3" H 1825 2700 50  0000 L CNN
-F 1 "100n" H 1825 2500 50  0000 L CNN
+F 1 "100nF" H 1825 2500 50  0000 L CNN
 F 2 "ultim8x8_libs:c_0805" H 1800 2600 50  0001 C CNN
 F 3 "" H 1800 2600 60  0001 C CNN
@@
 P 1250 6750
 F 0 "C4" H 1375 6725 50  0000 L CNN
-F 1 "47u,8V" H 1375 6625 50  0000 L CNN
+F 1 "47uF 20V" H 1375 6625 50  0000 L CNN
 F 2 "ultim8x8_libs:c_2917" H 1250 6700 50  0001 C CNN
 F 3 "" H 1250 6750 60  0001 C CNN

Commit message: revised layout, final. Gerbers ready for fab
Parts:
- U59: footprint ultim8x8_libs:APA102 -> ultim8x8_libs:APA102_U59
- U60: footprint ultim8x8_libs:APA102 -> ultim8x8_libs:APA102_U60
Changed lines of the file:
@@
 F 0 "U59" H 4100 1900 40  0000 C CNB
 F 1 "APA102" H 4100 1275 40  0000 C CNN
-F 2 "ultim8x8_libs:APA102" H 4000 2000 60  0001 C CNN
+F 2 "ultim8x8_libs:APA102_U59" H 4000 2000 60  0001 C CNN
 F 3 "" H 4100 1600 60  0001 C CNN
 F 4 "mfr_pn" H 4100 1600 60  0001 C CNN "manf#"
@@
 F 0 "U60" H 5300 1900 40  0000 C CNB
 F 1 "APA102" H 5300 1275 40  0000 C CNN
-F 2 "ultim8x8_libs:APA102" H 5200 2000 60  0001 C CNN
+F 2 "ultim8x8_libs:APA102_U60" H 5200 2000 60  0001 C CNN
 F 3 "" H 5300 1600 60  0001 C CNN
 F 4 "mfr_pn" H 5300 1600 60  0001 C CNN "manf#"
