File: kicad/ultim8x8.kicad_pcb (KiCad board)
At the start: 2 copper layers, 78 parts, among them P1 Input1, P2 Output1, P3 5V, P4 GND, P5 Input2, P6 Output2, U01 APA102, U02 APA102, U03 APA102, U04 APA102, U05 APA102, U06 APA102, U07 APA102, U08 APA102, U09 APA102, U10 APA102, U11 APA102, U12 APA102, U13 APA102, U14 APA102, U15 APA102, U16 APA102, U17 APA102, U18 APA102, U19 APA102, U20 APA102, U21 APA102, U22 APA102, U23 APA102, U24 APA102, U25 APA102, U26 APA102, U27 APA102, U28 APA102, U29 APA102, U30 APA102, U31 APA102, U32 APA102, U33 APA102, U34 APA102, U35 APA102, U36 APA102, U37 APA102, U38 APA102, U39 APA102, U40 APA102, U41 APA102, U42 APA102, U43 APA102, U44 APA102, U45 APA102, U46 APA102, U47 APA102, U48 APA102, U49 APA102, U50 APA102, U51 APA102, U52 APA102, U53 APA102, U54 APA102, U55 APA102, U56 APA102, U57 APA102, U58 APA102, U59 APA102, U60 APA102, U61 APA102, U62 APA102, U63 APA102, U64 APA102

Commit message: revised layout, final. Gerbers ready for fab
Parts:
- C1, C3: footprint TinyTiM_Libs:c_0805 -> ultim8x8_libs:c_0805
- C2: footprint TinyTiM_Libs:c_2917 -> ultim8x8_libs:c_2917
- C4: value 47uF 8V -> 47uF 20V; footprint TinyTiM_Libs:c_2917 -> ultim8x8_libs:c_2917
- L2: footprint TinyTiM_Lib:OSHW_6mm -> ultim8x8_libs:OSHW_6mm
- L3: footprint TinyTiM_Libs:logo_wyo_butterfly -> ultim8x8_libs:logo_wyo_butterfly
- L4: footprint TinyTiM_Libs:logo_MLlabs -> ultim8x8_libs:logo_MLlabs
- P1, P2, P5, P6: footprint TinyTiM_Libs:header_3pos_smd_male -> ultim8x8_libs:header_3pos_smd_male
- P3, P4: footprint TinyTiM_Libs:PowerIn_stud -> ultim8x8_libs:PowerIn_stud
- U05: footprint ultim8x8_libs:APA102 -> ultim8x8_libs:APA102_U05
- U06: footprint ultim8x8_libs:APA102 -> ultim8x8_libs:APA102_U06
- U11: footprint ultim8x8_libs:APA102 -> ultim8x8_libs:APA102_U11
- U12: footprint ultim8x8_libs:APA102 -> ultim8x8_libs:APA102_U12
- U19: footprint ultim8x8_libs:APA102 -> ultim8x8_libs:APA102_U19
- U38: footprint ultim8x8_libs:APA102 -> ultim8x8_libs:APA102_U38
- U43: footprint ultim8x8_libs:APA102 -> ultim8x8_libs:APA102_U43
- U53: footprint ultim8x8_libs:APA102 -> ultim8x8_libs:APA102_U53
- U54: footprint ultim8x8_libs:APA102 -> ultim8x8_libs:APA102_U54
- U59: footprint ultim8x8_libs:APA102 -> ultim8x8_libs:APA102_U59
- U60: footprint ultim8x8_libs:APA102 -> ultim8x8_libs:APA102_U60
- moved L4 0.36 mm to (44.7, 36.4)
- turned P4 to 180 degrees
Routing:
- net GND: track 104.6 -> 123.5 mm
- net /Row_A/CI_A: track 66.3 -> 74.3 mm
- net /Row_A/5V: track 584.2 -> 578.8 mm
- net /Row_A/DI_A: track 72.4 -> 67.3 mm
- net Net-(U52-Pad6): track 4.45 -> 3.22 mm
- net /Row_H/DO_H: track 82.9 -> 81.7 mm
