File: kicad/ultim8x8.sch (KiCad schematic (older format))
At the start: 9 parts, among them P1 Input1, P2 Output1, P3 5V, P4 GND, P5 Input2, P6 Output2

Commit message: UlTiM8x8 board layout complete. Gerbers ready. ULTiM_bus mockup
Parts:
- added L1: ULTiM8x8, ultim8x8_libs:logo_ultim8x8, symbol LOGO_1
- renumbered L101 to L2, L102 to L3, L103 to L4
Changed lines of the file:
@@
 encoding utf-8
 Sheet 1 9
-Title "UlTiM8 - Ultimate LED panel, using APA102"
+Title "ULTiM8x8 - Ultimate LED panel, using APA102"
 Date "2016-02-18"
 Rev "rev1"
@@
 01 31 04 0B 88 21 58 40 0C C1 02 62 08 16 10 43 B0 80 18 82 05 C4 10 2C 20 86 60 01 31 04 0B 88
 21 58 40 0C C1 02 62 08 16 10 43 B0 80 18 82 05 C4 10 2C 20 86 60 01 31 04 0B 88 21 58 40 0C C1
-02 62 7C 03 3D 79 5E 0E 30 13 47 E7 00 00 00 00 49 45 4E 44 AE 42 60 82 D1
+02 62 7C 03 3D 79 5E 0E 30 13 47 E7 00 00 00 00 49 45 4E 44 AE 42 60 82 91
 EndData
 $EndBitmap
@@
 	1350 1425 1600 1425
 $Comp
-L LOGO_1 L101
+L LOGO_1 L2
 U 1 1 511CD9F8
 P 1325 6600
-F 0 "L101" V 1425 6600 40  0000 C CNN
+F 0 "L2" V 1425 6600 40  0000 C CNN
 F 1 "OSHW" V 1225 6600 30  0000 C CNN
 F 2 "ultim8x8_libs:OSHW_6mm" H 1325 6755 30  0001 C CNN
@@
 $EndComp
 $Comp
-L LOGO_1 L102
+L LOGO_1 L3
 U 1 1 511CD9F5
 P 1675 6600
-F 0 "L102" V 1775 6600 40  0000 C CNN
+F 0 "L3" V 1775 6600 40  0000 C CNN
 F 1 "Wyolum" V 1575 6600 30  0000 C CNN
 F 2 "ultim8x8_libs:logo_wyo_butterfly" H 1600 6675 30  0001 C CNN
@@
 8 strips of 8 LEDs each (8x8)
 $Comp
-L LOGO_1 L103
+L LOGO_1 L4
 U 1 1 56C3209A
 P 2025 6600
-F 0 "L103" V 2125 6600 40  0000 C CNN
+F 0 "L4" V 2125 6600 40  0000 C CNN
 F 1 "Maniacal Labs" V 1925 6600 30  0000 C CNN
 F 2 "ultim8x8_libs:logo_MLlabs" H 1950 6675 30  0001 C CNN
@@
 60 BD D6 69 7C FA 84 4E 00 1C F3 6D BF C6 02 A0 13 00 C7 7C AB 8B FD F9 43 66 C3 B0 78 D8 F1 6E
 2F 80 9D 81 10 24 E6 C1 CF 81 0B 01 EC D4 00 18 4E AC 7F 37 5C 08 FB CB C7 8F 46 91 1C 94 52 FC
-EC F0 FD 0F 88 A0 E4 D1 04 AE BA DB 00 00 00 00 49 45 4E 44 AE 42 60 82 21
+EC F0 FD 0F 88 A0 E4 D1 04 AE BA DB 00 00 00 00 49 45 4E 44 AE 42 60 82 00
 EndData
 $EndBitmap
+$Comp
+L LOGO_1 L1
+U 1 1 56C5F837
+P 950 6600
+F 0 "L1" V 1050 6600 40  0000 C CNN
+F 1 "ULTiM8x8" V 850 6600 30  0000 C CNN
+F 2 "ultim8x8_libs:logo_ultim8x8" H 950 6755 30  0001 C CNN
+F 3 "" H 950 6600 60  0001 C CNN
+	1    950  6600
+	0    -1   -1   0
+$EndComp
 $EndSCHEMATC
