File: kicad_8x8_45/Row_A.sch (KiCad schematic (older format))
At the start: 10 parts, among them U01 APA102, U02 APA102, U03 APA102, U04 APA102, U05 APA102, U06 APA102, U07 APA102, U08 APA102

Commit message: angled LED version complete
Parts:
- C1: Field10 399-1168-1-ND -> (none); Field11 http://www.digikey.com/product-detail/en/C0805C104K3RACTU/3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 -> (none); Field4 CAP CER 0.1UF 25V 10% X7R 0805 -> (none); Field5 100nF, 25V -> (none); Field6 Surface Mount, MLCC -> (none); Field7 Kemet -> (none); Field8 C0805C104K3RACTU -> (none); Field9 Digikey -> (none); manf# (none) -> Value
- C2: footprint ultim8x8_libs:c_2917 -> ultim8x8_libs:C_1210_HandSoldering; Field10 PCE3606CT-ND -> (none); Field11 http://www.digikey.com/product-detail/en/EEF-CD0K470R/PCE36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 -> (none); Field4 CAP ALUM 47UF 8V 20% SMD -> (none); Field5 47u,8V -> (none); Field6 2917 (7343 Metric) -> (none); Field7 Panasonic Electronic Components -> (none); Field8 EEF-CD0K470R -> (none); Field9 Digikey -> (none)
Changed lines of the file:
@@
 F 2 "ultim8x8_libs:c_0805" H 1800 2600 50  0001 C CNN
 F 3 "" H 1800 2600 60  0001 C CNN
-F 4 "CAP CER 0.1UF 25V 10% X7R 0805" H 1800 2800 60  0001 L CNN "Field4"
-F 5 "100nF, 25V" H 1800 2900 60  0001 L CNN "Field5"
-F 6 "Surface Mount, MLCC" H 1800 3000 60  0001 L CNN "Field6"
-F 7 "Kemet" H 1800 3100 60  0001 L CNN "Field7"
-F 8 "C0805C104K3RACTU" H 1800 3200 60  0001 L CNN "Field8"
-F 9 "Digikey" H 1800 3300 60  0001 L CNN "Field9"
-F 10 "399-1168-1-ND" H 1800 3400 60  0001 L CNN "Field10"
-F 11 "http://www.digikey.com/product-detail/en/C0805C104K3RACTU/399-1168-1-ND/411443" H 1800 3500 60  0001 L CNN "Field11"
+F 4 "Value" H 1800 2600 60  0001 C CNN "manf#"
 	1    1800 2600
 	1    0    0    -1
@@
 F 0 "C2" H 1375 6725 40  0000 L CNB
 F 1 "47uF 20V" H 1375 6625 40  0000 L CNN
-F 2 "ultim8x8_libs:c_2917" H 1250 6700 50  0001 C CNN
+F 2 "ultim8x8_libs:C_1210_HandSoldering" H 1250 6700 50  0001 C CNN
 F 3 "" H 1250 6750 60  0001 C CNN
 F 4 "Value" H 1250 6750 60  0001 C CNN "manf#"
-F 5 "CAP ALUM 47UF 8V 20% SMD" H 1250 6950 60  0001 L CNN "Field4"
-F 6 "47u,8V" H 1250 7050 60  0001 L CNN "Field5"
-F 7 "2917 (7343 Metric)" H 1250 7150 60  0001 L CNN "Field6"
-F 8 "Panasonic Electronic Components" H 1250 7250 60  0001 L CNN "Field7"
-F 9 "EEF-CD0K470R" H 1250 7350 60  0001 L CNN "Field8"
-F 10 "Digikey" H 1250 7450 60  0001 L CNN "Field9"
-F 11 "PCE3606CT-ND" H 1250 7550 60  0001 L CNN "Field10"
-F 12 "http://www.digikey.com/product-detail/en/EEF-CD0K470R/PCE3606CT-ND/614442" H 1250 7650 60  0001 L CNN "Field11"
 	1    1250 6750
 	1    0    0    -1
