File: kicad_8x8_45/ultim_bus.kicad_pcb (KiCad board)
At the start: 2 copper layers, 198.1 x 48.3 mm, 154 parts, among them M1 MouseBite, M2 MouseBite, M3 MouseBite, M4 MouseBite, M5 MouseBite, M6 MouseBite, M8 MouseBite, P1 CONN_1, P10 CONN_1, P11 CONN_1, P12 CONN_1, P13 CONN_1, P14 CONN_1, P15 CONN_1, P16 CONN_1, P17 CONN_1, P18 CONN_1, P19 CONN_1, P2 CONN_1, P20 CONN_1, P21 CONN_1, P22 CONN_1, P23 CONN_1, P24 CONN_1, P3 CONN_1, P31 CONN_1, P32 CONN_1, P33 CONN_1, P34 CONN_1, P35 CONN_1, P36 CONN_1, P37 CONN_1, P38 CONN_1, P39 CONN_1, P4 CONN_1, P40 CONN_1, P41 CONN_1, P42 CONN_1, P5 CONN_1, P6 CONN_1, P67 CONN_1, P68 CONN_1, P69 CONN_1, P7 CONN_1, P8 CONN_1, P9 CONN_1

Commit message: ULTiM_bus redesign
Parts:
- removed the M5 at (35.6, 57.1)
- removed the M5 at (35.6, 44.5)
- removed the M6 at (96.5, 57.1)
- removed the M6 at (157.5, 57.1)
- removed the M6 at (157.5, 44.5)
- removed the M6 at (96.5, 44.5)
- removed the M8 at (218.4, 57.1)
- removed the M8 at (218.4, 44.5)
- removed the P10 at (157.5, 76.2)
- removed the P11 at (188.0, 76.2)
- removed the P2 at (81.3, 76.2)
- removed the P3 at (111.8, 76.2)
- removed the P31 at (50.8, 63.5)
- removed the P31 at (50.8, 50.8)
- removed the P32 at (66.0, 63.5)
- removed the P32 at (66.0, 50.8)
- removed the P34 at (96.5, 50.8)
- removed the P35 at (111.8, 63.5)
- removed the P35 at (111.8, 50.8)
- removed the P36 at (127.0, 63.5)
- removed the P36 at (127.0, 50.8)
- removed the P38 at (157.5, 50.8)
- removed the P39 at (172.7, 63.5)
- removed the P39 at (172.7, 50.8)
- removed the P40 at (188.0, 63.5)
- removed the P40 at (188.0, 50.8)
- removed the P6 at (203.2, 76.2)
- removed P67, P68, P69: CONN_1, ultim8x8_libs:Screw
- removed the P7 at (66.0, 76.2)
- added M10: MouseBite, ultim8x8_libs:mouse-bite-5.08mm-slot, F.Cu at (157.5, 53.3)
- added M11: MouseBite, ultim8x8_libs:mouse-bite-5.08mm-slot, F.Cu at (218.4, 53.3)
- added M15: MouseBite, ultim8x8_libs:mouse-bite-5.08mm-slot, F.Cu at (35.6, 68.6)
- added M16: MouseBite, ultim8x8_libs:mouse-bite-5.08mm-slot, F.Cu at (96.5, 68.6)
- added M17: MouseBite, ultim8x8_libs:mouse-bite-5.08mm-slot, F.Cu at (157.5, 68.6)
- added M18: MouseBite, ultim8x8_libs:mouse-bite-5.08mm-slot, F.Cu at (218.4, 68.6)
- added M8: MouseBite, ultim8x8_libs:mouse-bite-5.08mm-slot, F.Cu at (35.6, 53.3)
- added M9: MouseBite, ultim8x8_libs:mouse-bite-5.08mm-slot, F.Cu at (96.5, 53.3)
- added P12: CONN_1, ultim8x8_libs:Screw_SqPad, F.Cu at (203.2, 30.5)
- added P14: CONN_1, ultim8x8_libs:Screw, F.Cu at (35.6, 45.7)
- added P17: CONN_1, ultim8x8_libs:Screw, F.Cu at (81.3, 45.7)
- added P18: CONN_1, ultim8x8_libs:Screw, F.Cu at (96.5, 45.7)
- added P21: CONN_1, ultim8x8_libs:Screw, F.Cu at (142.2, 45.7)
- added P22: CONN_1, ultim8x8_libs:Screw, F.Cu at (157.5, 45.7)
- added P24: CONN_1, ultim8x8_libs:Screw_SqPad, F.Cu at (188.0, 45.7)
- added P25: CONN_1, ultim8x8_libs:Screw, F.Cu at (203.2, 45.7)
- added P28: CONN_1, ultim8x8_libs:Screw_SqPad, F.Cu at (50.8, 61.0)
- added P29: CONN_1, ultim8x8_libs:Screw_SqPad, F.Cu at (66.0, 61.0)
- added P32: CONN_1, ultim8x8_libs:Screw_SqPad, F.Cu at (111.8, 61.0)
- added P36: CONN_1, ultim8x8_libs:Screw_SqPad, F.Cu at (172.7, 61.0)
- added P40: CONN_1, ultim8x8_libs:Screw_SqPad, F.Cu at (35.6, 76.2)
- added P42: CONN_1, ultim8x8_libs:Screw, F.Cu at (66.0, 76.2)
- added P43: CONN_1, ultim8x8_libs:Screw_SqPad, F.Cu at (81.3, 76.2)
- added P44: CONN_1, ultim8x8_libs:Screw_SqPad, F.Cu at (96.5, 76.2)
- added P45: CONN_1, ultim8x8_libs:Screw, F.Cu at (111.8, 76.2)
- added P46: CONN_1, ultim8x8_libs:Screw, F.Cu at (127.0, 76.2)
- added P47: CONN_1, ultim8x8_libs:Screw_SqPad, F.Cu at (142.2, 76.2)
- added P48: CONN_1, ultim8x8_libs:Screw_SqPad, F.Cu at (157.5, 76.2)
- added P49: CONN_1, ultim8x8_libs:Screw, F.Cu at (172.7, 76.2)
- added P50: CONN_1, ultim8x8_libs:Screw, F.Cu at (188.0, 76.2)
- added P51: CONN_1, ultim8x8_libs:Screw_SqPad, F.Cu at (203.2, 76.2)
- M1, M2, M3, M4: footprint ultim8x8_libs:mouse-bite-2.54mm-slot -> ultim8x8_libs:mouse-bite-5.08mm-slot
- P1, P15, P16, P19, P20, P23, P33, P37, P4, P5, P8, P9: footprint ultim8x8_libs:Screw -> ultim8x8_libs:Screw_SqPad
- moved P41 154.5 mm to (50.8, 76.2)
- moved P5 88.9 mm to (96.5, 30.5)
- moved P4 76.2 mm to (81.3, 30.5)
- moved P8 64.7 mm to (142.2, 30.5)
- moved P9 54.9 mm to (157.5, 30.5)
- moved P1 48.2 mm to (35.6, 30.5)
- moved P33 46.8 mm to (127.0, 61.0)
- moved P37 46.8 mm to (188.0, 61.0)
- moved REF**1111 45.7 mm to (210.8, 25.4)
- moved REF**1111 45.7 mm to (149.9, 25.4)
- moved REF**1114 45.7 mm to (210.8, 29.2)
- moved REF**1114 45.7 mm to (149.9, 29.2)
- moved REF**1118 45.7 mm to (210.8, 34.3)
- moved REF**1118 45.7 mm to (149.9, 34.3)
- moved REF**112 45.7 mm to (88.9, 25.4)
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- renumbered L2 to L1, L11 to L10, L15 to L11, L14 to L12, L1 to L2, L7 to L3, L6 to L4, L7 to L6, L11 to L7, L10 to L8, M5 to M12, M5 to M13, M5 to M14, M5 to M6, M5 to M7, P21 to P10, P22 to P11, P24 to P13, P13 to P2, P42 to P26, P69 to P27, P14 to P3, P33 to P30, P34 to P31, P37 to P34, P38 to P35, P41 to P38, P42 to P39, P12 to P52, P17 to P6, P18 to P7
Connections:
- P10 pad 1: /ROW2 -> /ROW1
- P11 pad 1: /ROW2 -> /ROW1
- P13 pad 1: /ROW2 -> /ROW1
- P15 pad 1: /ROW2 -> /ROW31
- P16 pad 1: /ROW2 -> /ROW32
- P19 pad 1: /ROW2 -> /ROW32
- P2 pad 1: /ROW2 -> /ROW1
- P20 pad 1: /ROW2 -> /ROW33
- P23 pad 1: /ROW2 -> /ROW33
- P26 pad 1: /ROW3 -> /ROW34
- P27 pad 1: /ROW3 -> /ROW41
- P3 pad 1: /ROW2 -> /ROW1
- P30 pad 1: /ROW3 -> /ROW42
- P31 pad 1: /ROW3 -> /ROW42
- P33 pad 1: /ROW3 -> /ROW43
- P34 pad 1: /ROW3 -> /ROW43
- P35 pad 1: /ROW3 -> /ROW43
- P37 pad 1: /ROW3 -> /ROW44
- P38 pad 1: /ROW3 -> /ROW44
- P39 pad 1: /ROW3 -> /ROW44
- P41 pad 1: /ROW3 -> /ROW2
- P52 pad 1: /ROW1 -> /ROW2
- P6 pad 1: /ROW2 -> /ROW1
- P7 pad 1: /ROW2 -> /ROW1
- REF**1111111 pad 1: /ROW3 -> /ROW44
- REF**1111111 pad 1: /ROW3 -> /ROW34
- REF**11111110 pad 1: /ROW3 -> /ROW44
- REF**11111110 pad 1: /ROW3 -> /ROW34
- REF**1111112 pad 1: /ROW3 -> /ROW44
- REF**1111112 pad 1: /ROW3 -> /ROW34
- REF**1111113 pad 1: /ROW3 -> /ROW44
- REF**1111113 pad 1: /ROW3 -> /ROW34
- REF**1111114 pad 1: /ROW3 -> /ROW44
- REF**1111114 pad 1: /ROW3 -> /ROW34
- REF**1111115 pad 1: /ROW3 -> /ROW44
- REF**1111115 pad 1: /ROW3 -> /ROW34
- REF**1111116 pad 1: /ROW3 -> /ROW44
- REF**1111116 pad 1: /ROW3 -> /ROW34
- REF**1111117 pad 1: /ROW3 -> /ROW44
- REF**1111117 pad 1: /ROW3 -> /ROW34
- REF**1111118 pad 1: /ROW3 -> /ROW44
- REF**1111118 pad 1: /ROW3 -> /ROW34
Routing:
- net /ROW3: track 274.3 -> 0.00 mm
- net /ROW2: track 182.9 -> 30.5 mm
- net /ROW1: track 182.9 -> 30.5 mm
- net /ROW44: track 0.00 -> 2.54 mm
- net /ROW34: track 0.00 -> 2.54 mm
- added copper zone on B.Cu, net /ROW31
- added copper zone on F.Cu, net /ROW31
- added copper zone on B.Cu, net /ROW32
- added copper zone on F.Cu, net /ROW32
- added copper zone on B.Cu, net /ROW33
- added copper zone on F.Cu, net /ROW33
- added copper zone on B.Cu, net /ROW34
- added copper zone on F.Cu, net /ROW34
- added copper zone on B.Cu, net /ROW41
- added copper zone on F.Cu, net /ROW41
- added copper zone on B.Cu, net /ROW42
- added copper zone on F.Cu, net /ROW42
- added copper zone on B.Cu, net /ROW43
- added copper zone on F.Cu, net /ROW43
- added copper zone on B.Cu, net /ROW44
- added copper zone on F.Cu, net /ROW44
- removed copper zone on B.Cu, net /ROW3
- removed copper zone on F.Cu, net /ROW3
Other:
- board size 198.1 x 48.3 mm -> 198.1 x 55.9 mm
