File: kicad_8x8_45/ultim_bus.sch (KiCad schematic (older format))
At the start: 103 parts, among them M1 MouseBite, M10 MouseBite, M11 MouseBite, M12 MouseBite, M13 MouseBite, M14 MouseBite, M15 MouseBite, M16 MouseBite, M2 MouseBite, M3 MouseBite, M4 MouseBite, M5 MouseBite, M6 MouseBite, M7 MouseBite, M8 MouseBite, M9 MouseBite, P1 CONN_1, P10 CONN_1, P11 CONN_1, P12 CONN_1, P13 CONN_1, P14 CONN_1, P15 CONN_1, P16 CONN_1, P17 CONN_1, P18 CONN_1, P19 CONN_1, P2 CONN_1, P20 CONN_1, P21 CONN_1, P22 CONN_1, P23 CONN_1, P24 CONN_1, P25 CONN_1, P26 CONN_1, P27 CONN_1, P28 CONN_1, P29 CONN_1, P3 CONN_1, P30 CONN_1, P31 CONN_1, P32 CONN_1, P33 CONN_1, P34 CONN_1, P35 CONN_1, P36 CONN_1, P37 CONN_1, P38 CONN_1, P39 CONN_1, P4 CONN_1, P40 CONN_1, P41 CONN_1, P42 CONN_1, P43 CONN_1, P44 CONN_1, P45 CONN_1, P46 CONN_1, P47 CONN_1, P48 CONN_1, P49 CONN_1, P5 CONN_1, P50 CONN_1, P51 CONN_1, P52 CONN_1, P53 CONN_1, P54 CONN_1, P55 CONN_1, P56 CONN_1, P57 CONN_1, P58 CONN_1, P59 CONN_1, P6 CONN_1, P60 CONN_1, P61 CONN_1, P62 CONN_1, P63 CONN_1, P64 CONN_1, P65 CONN_1, P66 CONN_1, P67 CONN_1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

Commit message: ULTiM_bus redesign
Parts:
- removed L15, L16: ULTiM, ultim8x8_libs:logo_ultim8x8_small, symbol CONN_1
- removed L3, L4: OSHW, ultim8x8_libs:OSHW_6mm, symbol CONN_1
- removed P25, P26, P27, P28, P29, P30, P43, P44, P45, P46, P47, P48, P61, P62, P63, P64, P65, P66, P71: CONN_1, ultim8x8_libs:Screw, symbol CONN_1
- added M17, M18: MouseBite, ultim8x8_libs:mouse-bite-5.08mm-slot, symbol CONN_1
- M1, M10, M11, M15, M16, M2, M3, M4, M8, M9: footprint ultim8x8_libs:mouse-bite-2.54mm-slot -> ultim8x8_libs:mouse-bite-5.08mm-slot
- P1, P12, P4, P5, P8, P9: footprint ultim8x8_libs:Screw -> ultim8x8_libs:Screw_SqPad; manf# (none) -> Value
- P14: renamed from P13; manf# (none) -> Value
- P15: renamed from P14; footprint ultim8x8_libs:Screw -> ultim8x8_libs:Screw_SqPad; manf# (none) -> Value
- P16: renamed from P15; footprint ultim8x8_libs:Screw -> ultim8x8_libs:Screw_SqPad; manf# (none) -> Value
- P17: renamed from P16; manf# (none) -> Value
- P18: renamed from P17; manf# (none) -> Value
- P19: renamed from P18; footprint ultim8x8_libs:Screw -> ultim8x8_libs:Screw_SqPad; manf# (none) -> Value
- P20: renamed from P19; footprint ultim8x8_libs:Screw -> ultim8x8_libs:Screw_SqPad; manf# (none) -> Value
- P21: renamed from P20; manf# (none) -> Value
- P22: renamed from P21; manf# (none) -> Value
- P23: renamed from P22; footprint ultim8x8_libs:Screw -> ultim8x8_libs:Screw_SqPad; manf# (none) -> Value
- P24: renamed from P23; footprint ultim8x8_libs:Screw -> ultim8x8_libs:Screw_SqPad; manf# (none) -> Value
- P25: renamed from P24; manf# (none) -> Value
- P26: renamed from P68; manf# (none) -> Value
- P27: renamed from P31; manf# (none) -> Value
- P28: renamed from P32; footprint ultim8x8_libs:Screw -> ultim8x8_libs:Screw_SqPad; manf# (none) -> Value
- P29: renamed from P33; footprint ultim8x8_libs:Screw -> ultim8x8_libs:Screw_SqPad; manf# (none) -> Value
- P32: renamed from P36; footprint ultim8x8_libs:Screw -> ultim8x8_libs:Screw_SqPad; manf# (none) -> Value
- P33: renamed from P37; footprint ultim8x8_libs:Screw -> ultim8x8_libs:Screw_SqPad; manf# (none) -> Value
- P36: renamed from P40; footprint ultim8x8_libs:Screw -> ultim8x8_libs:Screw_SqPad; manf# (none) -> Value
- P37: renamed from P41; footprint ultim8x8_libs:Screw -> ultim8x8_libs:Screw_SqPad; manf# (none) -> Value
- P40: renamed from P49; footprint ultim8x8_libs:Screw -> ultim8x8_libs:Screw_SqPad; manf# (none) -> Value
- P41: renamed from P50; manf# (none) -> Value
- P42: renamed from P51; manf# (none) -> Value
- P43: renamed from P52; footprint ultim8x8_libs:Screw -> ultim8x8_libs:Screw_SqPad; manf# (none) -> Value
- P44: renamed from P53; footprint ultim8x8_libs:Screw -> ultim8x8_libs:Screw_SqPad; manf# (none) -> Value
- P45: renamed from P54; manf# (none) -> Value
- P46: renamed from P55; manf# (none) -> Value
- P47: renamed from P56; footprint ultim8x8_libs:Screw -> ultim8x8_libs:Screw_SqPad; manf# (none) -> Value
- P48: renamed from P57; footprint ultim8x8_libs:Screw -> ultim8x8_libs:Screw_SqPad; manf# (none) -> Value
- P49: renamed from P58; manf# (none) -> Value
- P50: renamed from P59; manf# (none) -> Value
- P51: renamed from P60; footprint ultim8x8_libs:Screw -> ultim8x8_libs:Screw_SqPad; manf# (none) -> Value
- renumbered L12 to L10, L13 to L11, L14 to L12, L5 to L3, L6 to L4, L7 to L5, L8 to L6, L9 to L7, L10 to L8, L11 to L9, P67 to P13, P34 to P30, P35 to P31, P38 to P34, P39 to P35, P42 to P38, P69 to P39, P70 to P52
Connections:
- net ROW4 is gone; now on net ROW2: P40.1, P41.1, P42.1, P43.1, P44.1, P45.1, P46.1, P47.1, P48.1, P49.1, P50.1, P51.1, P52.1
- net ROW2: no longer P14.1, P15.1, P16.1, P17.1, P18.1, P19.1, P20.1, P21.1, P22.1, P23.1, P24.1, P25.1, P26.1
- removed net ROW3: P27.1, P28.1, P29.1, P30.1, P31.1, P32.1, P33.1, P34.1, P35.1, P36.1, P37.1, P38.1, P39.1
- new net ROW31: P14.1, P15.1
- new net ROW32: P16.1, P17.1, P18.1, P19.1
- new net ROW33: P20.1, P21.1, P22.1, P23.1
- new net ROW34: P24.1, P25.1, P26.1
- new net ROW41: P27.1, P28.1
- new net ROW42: P29.1, P30.1, P31.1, P32.1
- new net ROW43: P33.1, P34.1, P35.1, P36.1
- new net ROW44: P37.1, P38.1, P39.1
- no-connect marks 51 -> 30
Other:
- moved on the sheet: M10, M11, M12, M13, M14, M15, M16, M8, M9, P14, P15, P16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
