File: kicad/kicad_8x8_45/ultim8x8.kicad_pcb (KiCad board)
At the start: 2 copper layers, 61 x 61 mm, 84 parts, among them P1 Input1, P10 DO_H, P11 5V, P12 GND, P2 Output1, P3 5V, P4 GND, P5 Input2, P6 Output2, P7 CI_A, P8 CO_H, P9 DI_A, U01 APA102, U02 APA102, U03 APA102, U04 APA102, U05 APA102, U06 APA102, U07 APA102, U08 APA102, U09 APA102, U10 APA102, U11 APA102, U12 APA102, U13 APA102, U14 APA102, U15 APA102, U16 APA102, U17 APA102, U18 APA102, U19 APA102, U20 APA102, U21 APA102, U22 APA102, U23 APA102, U24 APA102, U25 APA102, U26 APA102, U27 APA102, U28 APA102, U29 APA102, U30 APA102, U31 APA102, U32 APA102, U33 APA102, U34 APA102, U35 APA102, U36 APA102, U37 APA102, U38 APA102, U39 APA102, U40 APA102, U41 APA102, U42 APA102, U43 APA102, U44 APA102, U45 APA102, U46 APA102, U47 APA102, U48 APA102, U49 APA102, U50 APA102, U51 APA102, U52 APA102, U53 APA102, U54 APA102, U55 APA102, U56 APA102, U57 APA102, U58 APA102, U59 APA102, U60 APA102, U61 APA102, U62 APA102, U63 APA102, U64 APA102

Commit message: v2 of Feather carrier board
Connections:
- P2 pad 1: /DO_H -> /5V
- P2 pad 4: /5V -> /DO_H
- P5 pad 2: /DI_A -> /5V
- P5 pad 3: /5V -> /DI_A
Routing:
- net /DI_A: track 76.4 -> 79.4 mm
- net /DO_H: track 76.7 -> 79.2 mm
- net /5V: track 388.0 -> 387.3 mm
Changed lines of the file:
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@@
     (thickness 1.6002)
     (drawings 239)
-    (tracks 867)
+    (tracks 872)
     (zones 0)
     (modules 84)
@@
   )
   (setup
-    (last_trace_width 0.254)
+    (last_trace_width 0.508)
     (user_trace_width 0.2032)
     (user_trace_width 0.254)
@@
       (layerselection 0x010fc_80000001)
       (usegerberextensions true)
+      (usegerberattributes true)
       (excludeedgelayer true)
       (linewidth 0.254000)
@@
       (plotinvisibletext false)
       (padsonsilk false)
-      (subtractmaskfromsilk true)
+      (subtractmaskfromsilk false)
       (outputformat 1)
       (mirror false)
       (drillshape 0)
       (scaleselection 1)
-      (outputdirectory ultim8x8_images/))
+      (outputdirectory ultim8x8_gerber/))
   )
   (net 0 "")
@@
       (effects (font (size 1.016 1.016) (thickness 0.2032)) (justify mirror))
     )
-    (fp_text value Input2 (at -0.089803 3.681905 495) (layer B.SilkS)
+    (fp_text value Input2 (at 3.5023 0.089803 585) (layer B.SilkS)
       (effects (font (size 1.016 1.016) (thickness 0.2032)) (justify mirror))
     )
@@
       (net 116 /CI_A))
     (pad 3 thru_hole circle (at 1.27 -1.27 315) (size 1.397 1.397) (drill 1.016) (layers *.Cu *.Mask B.SilkS)
-      (net 114 /5V))
+      (net 115 /DI_A))
     (pad 4 thru_hole circle (at 1.27 1.27 315) (size 1.397 1.397) (drill 1.016) (layers *.Cu *.Mask B.SilkS)
       (net 1 GND))
     (pad 2 thru_hole circle (at -1.27 1.27 315) (size 1.397 1.397) (drill 1.016) (layers *.Cu *.Mask B.SilkS)
-      (net 115 /DI_A))
+      (net 114 /5V))
   )
   (module ultim8x8_libs:header_2x2pos_th_male (layer Back)
@@
       (effects (font (size 1.016 1.016) (thickness 0.2032)) (justify mirror))
     )
-    (fp_text value Output1 (at 0 3.937 45) (layer B.SilkS)
+    (fp_text value Output1 (at -3.681905 0.089803 315) (layer B.SilkS)
       (effects (font (size 1.016 1.016) (thickness 0.2032)) (justify mirror))
     )
@@
     (fp_line (start -2.794 -2.794) (end -2.794 2.794) (layer Dwgs.User) (width 0.254))
     (pad 1 thru_hole circle (at -1.27 -1.27 45) (size 1.397 1.397) (drill 1.016) (layers *.Cu *.Mask B.SilkS)
-      (net 117 /DO_H))
+      (net 114 /5V))
     (pad 3 thru_hole circle (at 1.27 -1.27 45) (size 1.397 1.397) (drill 1.016) (layers *.Cu *.Mask B.SilkS)
       (net 1 GND))
     (pad 4 thru_hole circle (at 1.27 1.27 45) (size 1.397 1.397) (drill 1.016) (layers *.Cu *.Mask B.SilkS)
-      (net 114 /5V))
+      (net 117 /DO_H))
     (pad 2 thru_hole circle (at -1.27 1.27 45) (size 1.397 1.397) (drill 1.016) (layers *.Cu *.Mask B.SilkS)
       (net 118 /CO_H))
@@
   (gr_circle (center 52.07 52.07) (end 50.165 52.07) (layer Dwgs.User) (width 0.254))
   (gr_circle (center 36.83 36.83) (end 34.925 36.83) (layer Dwgs.User) (width 0.254))
-  (gr_text "GND\n\n+5V" (at 61.722 42.418 45) (layer B.SilkS)
+  (gr_text "GND\n\n+5V" (at 55.626 40.386 315) (layer B.SilkS)
     (effects (font (size 0.762 1.016) (thickness 0.1905)) (justify right mirror))
   )
-  (gr_text "DO_H\n\nCO_H" (at 57.658 46.482 45) (layer B.SilkS)
+  (gr_text "DO_H\n\nCO_H" (at 63.754 48.641 315) (layer B.SilkS)
     (effects (font (size 0.762 1.016) (thickness 0.1905)) (justify left mirror))
   )
-  (gr_text "CI_A\n\nDI_A" (at 57.658 72.898 315) (layer B.SilkS)
+  (gr_text "CI_A\n\nDI_A" (at 63.754 70.993 45) (layer B.SilkS)
     (effects (font (size 0.762 1.016) (thickness 0.1905)) (justify left mirror))
   )
-  (gr_text "+5V\n\nGND" (at 61.722 76.962 315) (layer B.SilkS)
+  (gr_text "+5V\n\nGND" (at 55.626 78.994 45) (layer B.SilkS)
     (effects (font (size 0.762 1.016) (thickness 0.1905)) (justify right mirror))
   )
@@
   (segment (start 89.61269 79.729948) (end 89.61269 85.370052) (width 0.254) (layer Front) (net 113))
   (segment (start 89.61269 85.370052) (end 89.047006 85.935736) (width 0.254) (layer Front) (net 113) (status 20))
-  (segment (start 56.055735 48.084265) (end 59.69 44.45) (width 0.508) (layer Front) (net 114))
-  (segment (start 59.69 44.45) (end 61.486051 44.45) (width 0.508) (layer Front) (net 114))
-  (segment (start 55.455736 49.957056) (end 56.055735 49.357057) (width 0.508) (layer Front) (net 114))
-  (segment (start 56.055735 49.357057) (end 56.055735 48.084265) (width 0.508) (layer Front) (net 114))
-  (segment (start 65.197056 48.684264) (end 61.486051 44.973259) (width 0.635) (layer Front) (net 114))
-  (segment (start 61.486051 44.973259) (end 61.486051 44.45) (width 0.635) (layer Front) (net 114))
+  (segment (start 63.324265 71.295735) (end 59.69 74.93) (width 0.508) (layer Front) (net 114))
+  (segment (start 59.69 74.93) (end 57.893949 74.93) (width 0.508) (layer Front) (net 114))
+  (segment (start 63.924264 69.422944) (end 63.324265 70.022943) (width 0.508) (layer Front) (net 114))
+  (segment (start 63.324265 70.022943) (end 63.324265 71.295735) (width 0.508) (layer Front) (net 114))
+  (segment (start 57.893949 44.45) (end 57.893949 43.926741) (width 0.635) (layer Front) (net 114))
+  (segment (start 57.893949 43.926741) (end 54.182944 40.215736) (width 0.635) (layer Front) (net 114))
+  (segment (start 57.893949 74.93) (end 57.893949 74.406741) (width 0.635) (layer Front) (net 114))
+  (segment (start 57.893949 74.406741) (end 54.182944 70.695736) (width 0.635) (layer Front) (net 114))
   (segment (start 44.45 57.893949) (end 44.973259 57.893949) (width 0.635) (layer Front) (net 114))
   (segment (start 44.973259 57.893949) (end 48.684264 54.182944) (width 0.635) (layer Front) (net 114))
@@
   (segment (start 74.93 57.893949) (end 75.453259 57.893949) (width 0.635) (layer Front) (net 114))
   (segment (start 75.453259 57.893949) (end 79.164264 54.182944) (width 0.635) (layer Front) (net 114))
-  (segment (start 61.486051 74.93) (end 61.486051 76.726051) (width 0.635) (layer Front) (net 114))
-  (segment (start 61.486051 76.726051) (end 63.924264 79.164264) (width 0.635) (layer Front) (net 114))
-  (segment (start 65.197056 79.164264) (end 63.924264 79.164264) (width 0.635) (layer Front) (net 114))
   (segment (start 48.684264 84.662944) (end 45.165944 84.662944) (width 0.635) (layer Back) (net 114) (status 10))
   (segment (start 45.165944 84.662944) (end 44.45 83.947) (width 0.635) (layer Back) (net 114))
@@
   (segment (start 32.595736 83.672994) (end 32.595736 83.814416) (width 0.635) (layer Front) (net 114) (status 30))
   (segment (start 32.595736 83.814416) (end 33.444264 84.662944) (width 0.635) (layer Front) (net 114) (status 30))
+  (segment (start 52.07 61.486051) (end 55.651513 61.486051) (width 0.254) (layer Back) (net 115))
+  (segment (start 55.651513 61.486051) (end 59.055 64.889538) (width 0.254) (layer Back) (net 115))
+  (segment (start 59.055 64.889538) (end 59.055 71.755) (width 0.254) (layer Back) (net 115))
+  (segment (start 59.055 71.755) (end 58.42 72.39) (width 0.254) (layer Back) (net 115))
+  (segment (start 58.42 72.39) (end 58.42 73.66) (width 0.254) (layer Back) (net 115))
+  (segment (start 58.42 73.66) (end 59.69 74.93) (width 0.254) (layer Back) (net 115))
+  (segment (start 59.69 74.93) (end 61.486051 74.93) (width 0.254) (layer Back) (net 115))
   (segment (start 44.45 61.486051) (end 32.112949 61.486051) (width 0.254) (layer Back) (net 115))
   (segment (start 32.112949 61.486051) (end 31.574252 62.024748) (width 0.254) (layer Back) (net 115))
@@
   (segment (start 33.481757 87.803243) (end 31.57678 87.803243) (width 0.254) (layer Back) (net 115))
   (segment (start 44.45 61.486051) (end 52.07 61.486051) (width 0.254) (layer Back) (net 115))
-  (segment (start 52.07 61.486051) (end 55.651513 61.486051) (width 0.254) (layer Back) (net 115))
   (segment (start 52.07 67.31) (end 52.07 61.486051) (width 0.254) (layer Back) (net 115))
-  (segment (start 55.651513 61.486051) (end 57.893949 63.728487) (width 0.254) (layer Back) (net 115))
-  (segment (start 57.893949 63.728487) (end 57.893949 74.93) (width 0.254) (layer Back) (net 115))
   (segment (start 33.444264 89.047006) (end 32.200501 87.803243) (width 0.254) (layer Front) (net 115) (status 10))
   (segment (start 32.200501 87.803243) (end 31.57678 87.803243) (width 0.254) (layer Front) (net 115))
@@
   (via (at 32.385008 86.977723) (size 0.889) (drill 0.635) (layers Front Back) (net 116))
   (segment (start 34.575635 87.915635) (end 33.637723 86.977723) (width 0.254) (layer Front) (net 116) (status 10))
-  (segment (start 57.893949 44.45) (end 57.893949 53.448949) (width 0.254) (layer Back) (net 117))
+  (segment (start 57.893949 46.246051) (end 59.69 44.45) (width 0.254) (layer Back) (net 117))
+  (segment (start 59.69 44.45) (end 61.486051 44.45) (width 0.254) (layer Back) (net 117))
+  (segment (start 57.893949 53.448949) (end 57.893949 46.246051) (width 0.254) (layer Back) (net 117))
   (segment (start 57.893949 53.448949) (end 65.931051 61.486051) (width 0.254) (layer Back) (net 117))
   (segment (start 65.931051 61.486051) (end 67.31 61.486051) (width 0.254) (layer Back) (net 117))

Commit message: clean up
Routing:
- net /5V: track 387.3 -> 687.9 mm
- net /CO_H: track 81.6 -> 80.9 mm
Other:
- board text added: "+5V CI_A"
- board text added: "+5V CO_H"
- board text added: "CLK IN"
- board text added: "CLK OUT"
- board text added: "DAT IN"
- board text added: "DAT OUT"
- board text added: "GND DI_A"
- board text added: "GND DO_H"
- board text removed: "CLK_IN"
- board text removed: "CLK_OUT"
- board text removed: "DAT_IN"
- board text removed: "DAT_OUT"
- board text removed: "DO_H CO_H"
- board text removed: "GND +5V"
