File: kicad/kicad_8x8_45/ultim8x8.sch (KiCad schematic (older format))
At the start: 16 parts, among them P1 Input1, P10 DO_H, P11 5V, P12 GND, P2 Output1, P3 5V, P4 GND, P5 Input2, P6 Output2, P7 CI_A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

Commit message: board outline changed. upgraded 3 pin headers to 4 pins
Parts:
- P1, P2, P5, P6: footprint ultim8x8_libs:header_3pos_th_male -> ultim8x8_libs:header_2x2pos_th_male; symbol CONN_3 -> CONN4_S; manf# (none) -> Value
Connections:
- net 5V: now also P1.4 (P4), P2.4 (P4), P5.3 (P3), P6.2 (P2)
- net CI_A: now also P5.1 (P1); no longer P5.2 (P2)
- net CO_H: now also P6.4 (P4); no longer P6.2 (P2)
- net DI_A: now also P5.2 (P2); no longer P5.3 (P3)
- net GND: now also P5.4 (P4); no longer P5.1 (P1)
Changed lines of the file:
@@
 Text Label 2225 4750 0    60   ~ 0
 5V
-Text Label 1550 2100 2    40   ~ 0
+Text Label 1550 2200 2    40   ~ 0
 DI_A
-Wire Wire Line
-	1350 2100 1600 2100
-Text Label 1550 2300 2    40   ~ 0
+Text Label 1550 2400 2    40   ~ 0
 GND
 Wire Wire Line
 	1350 2300 1550 2300
+Text Label 1800 2300 0    40   ~ 0
+DO_H
 Text Label 1800 2100 0    40   ~ 0
-DO_H
-Wire Wire Line
-	1750 2100 2000 2100
-Text Label 1800 2300 0    40   ~ 0
 GND
 Wire Wire Line
-	2000 2300 1800 2300
+	1750 2300 2000 2300
 Text Label 1550 1525 2    40   ~ 0
 DI_A
@@
 	1800 2200 2000 2200
 Wire Wire Line
-	1550 2200 1350 2200
-Text Label 1800 2200 0    40   ~ 0
+	1350 2200 1600 2200
+Text Label 1800 2400 0    40   ~ 0
 CO_H
-Text Label 1550 2200 2    40   ~ 0
+Text Label 1525 2100 2    40   ~ 0
 CI_A
 Wire Wire Line
@@
 Connection ~ 975  5250
 $Comp
-L CONN_3 P1
+L CONN4_S P1
 U 1 1 56C0E218
-P 1000 1425
-F 0 "P1" H 1025 1225 40  0000 C CNB
+P 1000 1375
+F 0 "P1" H 1000 1125 40  0000 C CNB
 F 1 "Input1" H 1000 1625 40  0000 C CNN
-F 2 "ultim8x8_libs:header_3pos_th_male" H 1000 1375 60  0001 C CNN
-F 3 "" H 1000 1375 60  0000 C CNN
-F 4 "CONN HEADER 50POS .100\" SGL GOLD" H 1000 1475 60  0001 L CNN "Field4"
-F 5 "Header, Unshrouded, Male pin," H 1000 1575 60  0001 L CNN "Field5"
-F 6 "0.1\"" H 1000 1675 60  0001 L CNN "Field6"
-	1    1000 1425
+F 2 "ultim8x8_libs:header_2x2pos_th_male" H 1000 1325 60  0001 C CNN
+F 3 "" H 1000 1325 60  0000 C CNN
+F 4 "Value" H 1000 1375 60  0001 C CNN "manf#"
+F 5 "CONN HEADER 50POS .100\" SGL GOLD" H 1000 1425 60  0001 L CNN "Field4"
+F 6 "Header, Unshrouded, Male pin," H 1000 1525 60  0001 L CNN "Field5"
+F 7 "0.1\"" H 1000 1625 60  0001 L CNN "Field6"
+	1    1000 1375
 	-1   0    0    1
 $EndComp
 $Comp
-L CONN_3 P2
+L CONN4_S P2
 U 1 1 56C0F3D8
-P 2350 1425
-F 0 "P2" H 2350 1225 40  0000 C CNB
+P 2350 1375
+F 0 "P2" H 2350 1125 40  0000 C CNB
 F 1 "Output1" H 2350 1625 40  0000 C CNN
-F 2 "ultim8x8_libs:header_3pos_th_male" H 2350 1375 60  0001 C CNN
-F 3 "" H 2350 1375 60  0000 C CNN
-F 4 "CONN HEADER 50POS .100\" SGL GOLD" H 2350 1475 60  0001 L CNN "Field4"
-F 5 "Header, Unshrouded, Male pin," H 2350 1575 60  0001 L CNN "Field5"
-F 6 "0.1\"" H 2350 1675 60  0001 L CNN "Field6"
-	1    2350 1425
+F 2 "ultim8x8_libs:header_2x2pos_th_male" H 2350 1325 60  0001 C CNN
+F 3 "" H 2350 1325 60  0000 C CNN
+F 4 "Value" H 2350 1375 60  0001 C CNN "manf#"
+F 5 "CONN HEADER 50POS .100\" SGL GOLD" H 2350 1425 60  0001 L CNN "Field4"
+F 6 "Header, Unshrouded, Male pin," H 2350 1525 60  0001 L CNN "Field5"
+F 7 "0.1\"" H 2350 1625 60  0001 L CNN "Field6"
+	1    2350 1375
 	1    0    0    1
 $EndComp
 $Comp
-L CONN_3 P5
+L CONN4_S P5
 U 1 1 56C10A4A
-P 1000 2200
+P 1000 2250
 F 0 "P5" H 1000 2000 40  0000 C CNB
-F 1 "Input2" H 1000 2400 40  0000 C CNN
-F 2 "ultim8x8_libs:header_3pos_th_male" H 1000 2150 60  0001 C CNN
-F 3 "" H 1000 2150 60  0000 C CNN
-F 4 "CONN HEADER 50POS .100\" SGL GOLD" H 1000 2250 60  0001 L CNN "Field4"
-F 5 "Header, Unshrouded, Male pin," H 1000 2350 60  0001 L CNN "Field5"
-F 6 "0.1\"" H 1000 2450 60  0001 L CNN "Field6"
-	1    1000 2200
-	-1   0    0    1
-$EndComp
-$Comp
-L CONN_3 P6
+F 1 "Input2" H 1000 2500 40  0000 C CNN
+F 2 "ultim8x8_libs:header_2x2pos_th_male" H 1000 2200 60  0001 C CNN
+F 3 "" H 1000 2200 60  0000 C CNN
+F 4 "Value" H 1000 2250 60  0001 C CNN "manf#"
+F 5 "CONN HEADER 50POS .100\" SGL GOLD" H 1000 2300 60  0001 L CNN "Field4"
+F 6 "Header, Unshrouded, Male pin," H 1000 2400 60  0001 L CNN "Field5"
+F 7 "0.1\"" H 1000 2500 60  0001 L CNN "Field6"
+	1    1000 2250
+	-1   0    0    -1
+$EndComp
+$Comp
+L CONN4_S P6
 U 1 1 56C121A8
-P 2350 2200
+P 2350 2250
 F 0 "P6" H 2350 2000 40  0000 C CNB
-F 1 "Output2" H 2350 2400 40  0000 C CNN
-F 2 "ultim8x8_libs:header_3pos_th_male" H 2350 2150 60  0001 C CNN
-F 3 "" H 2350 2150 60  0000 C CNN
-F 4 "CONN HEADER 50POS .100\" SGL GOLD" H 2350 2250 60  0001 L CNN "Field4"
-F 5 "Header, Unshrouded, Male pin," H 2350 2350 60  0001 L CNN "Field5"
-F 6 "0.1\"" H 2350 2450 60  0001 L CNN "Field6"
-	1    2350 2200
-	1    0    0    1
+F 1 "Output2" H 2350 2500 40  0000 C CNN
+F 2 "ultim8x8_libs:header_2x2pos_th_male" H 2350 2200 60  0001 C CNN
+F 3 "" H 2350 2200 60  0000 C CNN
+F 4 "Value" H 2350 2250 60  0001 C CNN "manf#"
+F 5 "CONN HEADER 50POS .100\" SGL GOLD" H 2350 2300 60  0001 L CNN "Field4"
+F 6 "Header, Unshrouded, Male pin," H 2350 2400 60  0001 L CNN "Field5"
+F 7 "0.1\"" H 2350 2500 60  0001 L CNN "Field6"
+	1    2350 2250
+	1    0    0    -1
 $EndComp
 Text Label 6450 6500 2    60   ~ 0
@@
 Text Notes 700  3950 0    60   ~ 12
 POWER INPUT POSTS
-Text Notes 2000 2700 0    60   ~ 12
+Text Notes 2000 2875 0    60   ~ 12
 DATA/CLK\nOUTPUTS
-Text Notes 900  2700 0    60   ~ 12
+Text Notes 900  2875 0    60   ~ 12
 DATA/CLK\nINPUTS
 Text Notes 2850 900  0    60   ~ 12
@@
 	1600 1425 1600 1200
 Wire Wire Line
-	1750 1975 1750 2100
-Wire Wire Line
-	1600 2100 1600 1975
+	1750 1975 1750 2300
+Wire Wire Line
+	1600 2200 1600 1975
+Wire Wire Line
+	1550 1225 1350 1225
+Wire Wire Line
+	1800 1225 2000 1225
+Wire Wire Line
+	1800 2400 2000 2400
+Wire Wire Line
+	1550 2400 1350 2400
+Text Label 1550 2300 2    40   ~ 0
+5V
+Text Label 1800 2200 0    40   ~ 0
+5V
+Text Label 1800 1225 0    40   ~ 0
+5V
+Text Label 1550 1225 2    40   ~ 0
+5V
+Wire Wire Line
+	1800 2100 2000 2100
+Wire Wire Line
+	1525 2100 1350 2100
 $EndSCHEMATC

Commit message: v2 of Feather carrier board
Connections:
- net 5V: now also P2.1 (P1), P5.2 (P2); no longer P2.4 (P4), P5.3 (P3)
- net DI_A: now also P5.3 (P3); no longer P5.2 (P2)
- net DO_H: now also P2.4 (P4); no longer P2.1 (P1)
Changed lines of the file:
@@
 Text Label 2225 4750 0    60   ~ 0
 5V
-Text Label 1550 2200 2    40   ~ 0
+Text Label 1550 2300 2    40   ~ 0
 DI_A
 Text Label 1550 2400 2    40   ~ 0
 GND
 Wire Wire Line
-	1350 2300 1550 2300
+	1600 2300 1350 2300
 Text Label 1800 2300 0    40   ~ 0
 DO_H
 Text Label 1800 2100 0    40   ~ 0
 GND
-Wire Wire Line
-	1750 2300 2000 2300
 Text Label 1550 1525 2    40   ~ 0
 DI_A
-Text Label 1800 1525 0    40   ~ 0
+Text Label 1800 1225 0    40   ~ 0
 DO_H
 Wire Wire Line
@@
 Text Label 1800 1425 0    40   ~ 0
 CO_H
-Wire Wire Line
-	1800 2200 2000 2200
-Wire Wire Line
-	1350 2200 1600 2200
 Text Label 1800 2400 0    40   ~ 0
 CO_H
@@
 60 BD D6 69 7C FA 84 4E 00 1C F3 6D BF C6 02 A0 13 00 C7 7C AB 8B FD F9 43 66 C3 B0 78 D8 F1 6E
 2F 80 9D 81 10 24 E6 C1 CF 81 0B 01 EC D4 00 18 4E AC 7F 37 5C 08 FB CB C7 8F 46 91 1C 94 52 FC
-EC F0 FD 0F 88 A0 E4 D1 04 AE BA DB 00 00 00 00 49 45 4E 44 AE 42 60 82 21
+EC F0 FD 0F 88 A0 E4 D1 04 AE BA DB 00 00 00 00 49 45 4E 44 AE 42 60 82
 EndData
 $EndBitmap
@@
 04 25 3C 11 11 B1 04 25 3C 11 11 B1 04 25 3C 11 11 B1 04 25 3C 11 11 B1 04 25 3C 11 11 B1 04 25
 3C 11 11 B1 04 25 3C 11 11 B1 04 25 3C 11 11 B1 04 25 3C 11 11 B1 04 25 3C 11 11 B1 04 25 3C 11
-11 B1 04 25 3C 11 11 B1 84 FF 0F 4A 0D 97 B8 B1 77 E7 67 00 00 00 00 49 45 4E 44 AE 42 60 82 00
+11 B1 04 25 3C 11 11 B1 84 FF 0F 4A 0D 97 B8 B1 77 E7 67 00 00 00 00 49 45 4E 44 AE 42 60 82
 EndData
 $EndBitmap
@@
 	1750 1975 1750 2300
 Wire Wire Line
-	1600 2200 1600 1975
+	1600 1975 1600 2300
 Wire Wire Line
 	1550 1225 1350 1225
@@
 Wire Wire Line
 	1550 2400 1350 2400
-Text Label 1550 2300 2    40   ~ 0
+Text Label 1525 2200 2    40   ~ 0
 5V
 Text Label 1800 2200 0    40   ~ 0
 5V
-Text Label 1800 1225 0    40   ~ 0
+Text Label 1800 1525 0    40   ~ 0
 5V
 Text Label 1550 1225 2    40   ~ 0
@@
 Wire Wire Line
 	1525 2100 1350 2100
+Wire Wire Line
+	1750 2300 2000 2300
+Wire Wire Line
+	1525 2200 1350 2200
+Wire Wire Line
+	1800 2200 2000 2200
 $EndSCHEMATC

Commit message: clean up of all kicad project folders
Parts:
- L1: symbol LOGO_1 -> LOGO_U88; manf# (none) -> mfr_pn
- L2: symbol LOGO_1 -> OSHW; manf# (none) -> mfr_pn
- L3: symbol LOGO_1 -> LOGO_WL; manf# (none) -> mfr_pn
- L4: symbol LOGO_1 -> LOGO_ML; manf# (none) -> mfr_pn
Other:
- moved on the sheet: L4
