File: kicad/feather_v2/feather_v2.kicad_pcb (KiCad board)
At the start: 2 copper layers, 50.8 x 22.9 mm, 9 parts, among them P1 Maniacal Labs, P10 WyoLum, P2 Screw, P3 Screw, P6 Input, P7 Output, P8 Feather_M0

Commit message: clean up of all kicad project folders
Parts:
- added L3: OSHW, feather_v2:OSHW_6mm, B.Cu at (101.6, 101.6)
- L1: renamed from P10; value WyoLum -> LOGO_WL
- L2: renamed from P1; value Maniacal Labs -> LOGO_ML
- renumbered P2 to M1, P3 to M2
Changed lines of the file:
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@@
-(kicad_pcb (version 4) (host pcbnew 4.0.5-e0-6337~49~ubuntu16.04.1)
+(kicad_pcb (version 4) (host pcbnew 4.0.6-e0-6349~53~ubuntu16.04.1)
   (general
     (links 17)
@@
     (tracks 44)
     (zones 0)
-    (modules 9)
+    (modules 10)
     (nets 7)
   )
   (page A4)
   (layers
-    (0 F.Cu signal)
-    (31 B.Cu signal)
+    (0 F.Cu signal hide)
+    (31 B.Cu signal hide)
     (32 B.Adhes user)
     (33 F.Adhes user)
@@
       (layerselection 0x010f0_80000001)
       (usegerberextensions true)
+      (usegerberattributes true)
       (excludeedgelayer true)
       (linewidth 0.101600)
@@
   (module feather_v2:logo_MLlabs_small (layer F.Cu)
     (at 107.95 101.6 90)
-    (fp_text reference P1 (at 0 0 90) (layer F.SilkS) hide
-      (effects (font (size 1.016 1.016) (thickness 0.1524)))
-    )
-    (fp_text value "Maniacal Labs" (at 0.75 0 90) (layer F.SilkS) hide
+    (fp_text reference L2 (at 0 0 90) (layer F.SilkS) hide
+      (effects (font (size 1.016 1.016) (thickness 0.1524)))
+    )
+    (fp_text value LOGO_ML (at 0.75 0 90) (layer F.SilkS) hide
       (effects (font (size 1.016 1.016) (thickness 0.1524)))
     )
@@
   (module feather_v2:logo_wyo_butterfly_small (layer F.Cu)
     (at 99.187 101.6 45)
-    (fp_text reference P10 (at 0 -2 45) (layer F.SilkS) hide
-      (effects (font (size 1.016 1.016) (thickness 0.1524)))
-    )
-    (fp_text value WyoLum (at 0 1.5 45) (layer F.SilkS) hide
+    (fp_text reference L1 (at 0 -2 45) (layer F.SilkS) hide
+      (effects (font (size 1.016 1.016) (thickness 0.1524)))
+    )
+    (fp_text value LOGO_WL (at 0 1.5 45) (layer F.SilkS) hide
       (effects (font (size 1.016 1.016) (thickness 0.1524)))
     )
@@
   (module feather_v2:Screw_NPTH (layer F.Cu)
     (at 109.22 93.98)
-    (fp_text reference P2 (at 0 -1.5875) (layer F.SilkS) hide
+    (fp_text reference M1 (at 0 -1.5875) (layer F.SilkS) hide
       (effects (font (size 1.016 1.016) (thickness 0.1524)))
     )
@@
   (module feather_v2:Screw_NPTH (layer F.Cu)
     (at 93.98 109.22)
-    (fp_text reference P3 (at 0 -1.5875) (layer F.SilkS) hide
+    (fp_text reference M2 (at 0 -1.5875) (layer F.SilkS) hide
       (effects (font (size 1.016 1.016) (thickness 0.1524)))
     )
@@
     )
   )
+  (module feather_v2:OSHW_6mm (layer B.Cu)
+    (at 101.6 101.6 270)
+    (fp_text reference L3 (at 0 -1.016 270) (layer B.SilkS) hide
+      (effects (font (size 1.016 1.016) (thickness 0.2032)) (justify mirror))
+    )
+    (fp_text value OSHW (at 0 0.127 270) (layer B.SilkS) hide
+      (effects (font (size 1.016 1.016) (thickness 0.2032)) (justify mirror))
+    )
+    (fp_text user OpenHardware (at 0 -4.191 270) (layer B.SilkS)
+      (effects (font (size 0.762 0.6096) (thickness 0.127)) (justify mirror))
+    )
+    (fp_poly (pts (xy -2.02438 -2.99974) (xy -1.98882 -2.97942) (xy -1.91008 -2.93116) (xy -1.79832 -2.8575)
+      (xy -1.66624 -2.77114) (xy -1.53416 -2.6797) (xy -1.42494 -2.60858) (xy -1.34874 -2.55778)
+      (xy -1.31826 -2.54) (xy -1.30048 -2.54762) (xy -1.23698 -2.5781) (xy -1.14808 -2.62382)
+      (xy -1.09474 -2.65176) (xy -1.01092 -2.68732) (xy -0.96774 -2.69494) (xy -0.96266 -2.68478)
+      (xy -0.93218 -2.62128) (xy -0.88392 -2.51206) (xy -0.82042 -2.36728) (xy -0.74676 -2.1971)
+      (xy -0.67056 -2.01422) (xy -0.59182 -1.8288) (xy -0.51816 -1.651) (xy -0.45466 -1.49098)
+      (xy -0.40132 -1.3589) (xy -0.36576 -1.27) (xy -0.35306 -1.2319) (xy -0.35814 -1.22174)
+      (xy -0.39878 -1.1811) (xy -0.47244 -1.12776) (xy -0.62992 -0.99822) (xy -0.7874 -0.80518)
+      (xy -0.88138 -0.5842) (xy -0.9144 -0.33782) (xy -0.88646 -0.10922) (xy -0.79756 0.10922)
+      (xy -0.64516 0.3048) (xy -0.45974 0.45212) (xy -0.24384 0.54356) (xy 0 0.57404)
+      (xy 0.23114 0.54864) (xy 0.45466 0.45974) (xy 0.65278 0.30988) (xy 0.7366 0.21336)
+      (xy 0.8509 0.01524) (xy 0.9144 -0.19812) (xy 0.92202 -0.254) (xy 0.91186 -0.48768)
+      (xy 0.84328 -0.7112) (xy 0.71882 -0.91186) (xy 0.54864 -1.07696) (xy 0.52578 -1.0922)
+      (xy 0.44704 -1.15316) (xy 0.3937 -1.1938) (xy 0.35052 -1.22682) (xy 0.65024 -1.94564)
+      (xy 0.6985 -2.05994) (xy 0.77978 -2.25806) (xy 0.8509 -2.4257) (xy 0.90932 -2.56032)
+      (xy 0.94996 -2.65176) (xy 0.96774 -2.68732) (xy 0.96774 -2.68986) (xy 0.99568 -2.69494)
+      (xy 1.04902 -2.67462) (xy 1.15062 -2.62636) (xy 1.21666 -2.5908) (xy 1.29286 -2.55524)
+      (xy 1.32842 -2.54) (xy 1.35636 -2.55778) (xy 1.43002 -2.6035) (xy 1.5367 -2.67462)
+      (xy 1.66624 -2.76352) (xy 1.78816 -2.84734) (xy 1.89992 -2.921) (xy 1.9812 -2.97434)
+      (xy 2.02184 -2.99466) (xy 2.02692 -2.99466) (xy 2.06248 -2.97434) (xy 2.12852 -2.921)
+      (xy 2.22504 -2.82956) (xy 2.36474 -2.6924) (xy 2.38506 -2.66954) (xy 2.49936 -2.55524)
+      (xy 2.5908 -2.45872) (xy 2.6543 -2.3876) (xy 2.67716 -2.35712) (xy 2.67716 -2.35712)
+      (xy 2.65684 -2.31902) (xy 2.6035 -2.2352) (xy 2.52984 -2.1209) (xy 2.4384 -1.98882)
+      (xy 2.19964 -1.64338) (xy 2.33172 -1.31572) (xy 2.37236 -1.21666) (xy 2.42316 -1.09474)
+      (xy 2.46126 -1.00838) (xy 2.47904 -0.97028) (xy 2.5146 -0.95758) (xy 2.6035 -0.93726)
+      (xy 2.73304 -0.90932) (xy 2.88798 -0.88138) (xy 3.0353 -0.85344) (xy 3.16738 -0.82804)
+      (xy 3.2639 -0.81026) (xy 3.30708 -0.80264) (xy 3.31724 -0.79502) (xy 3.3274 -0.7747)
+      (xy 3.33248 -0.72898) (xy 3.33502 -0.6477) (xy 3.33756 -0.5207) (xy 3.33756 -0.33782)
+      (xy 3.33756 -0.3175) (xy 3.33502 -0.14224) (xy 3.33248 -0.00254) (xy 3.3274 0.0889)
+      (xy 3.32232 0.12446) (xy 3.32232 0.12446) (xy 3.27914 0.13462) (xy 3.18516 0.15494)
+      (xy 3.05308 0.18034) (xy 2.8956 0.21082) (xy 2.88544 0.21336) (xy 2.72796 0.24384)
+      (xy 2.59334 0.27178) (xy 2.5019 0.2921) (xy 2.4638 0.3048) (xy 2.45364 0.31496)
+      (xy 2.42316 0.37846) (xy 2.37744 0.47498) (xy 2.3241 0.59436) (xy 2.2733 0.71882)
+      (xy 2.23012 0.83058) (xy 2.19964 0.9144) (xy 2.18948 0.9525) (xy 2.18948 0.9525)
+      (xy 2.21488 0.9906) (xy 2.26822 1.07188) (xy 2.34442 1.18618) (xy 2.4384 1.3208)
+      (xy 2.44348 1.33096) (xy 2.53492 1.46304) (xy 2.60858 1.57734) (xy 2.65684 1.65862)
+      (xy 2.67716 1.69418) (xy 2.67462 1.69672) (xy 2.64668 1.73482) (xy 2.5781 1.81102)
+      (xy 2.48158 1.91262) (xy 2.36474 2.032) (xy 2.32664 2.06756) (xy 2.1971 2.19456)
+      (xy 2.10566 2.27838) (xy 2.04978 2.32156) (xy 2.02438 2.33172) (xy 2.02184 2.33172)
+      (xy 1.9812 2.30632) (xy 1.89738 2.25044) (xy 1.78308 2.17424) (xy 1.64846 2.0828)
+      (xy 1.6383 2.07518) (xy 1.50622 1.98374) (xy 1.39446 1.91008) (xy 1.31572 1.85674)
+      (xy 1.28016 1.83642) (xy 1.27508 1.83642) (xy 1.2192 1.85166) (xy 1.12522 1.88468)
+      (xy 1.00838 1.9304) (xy 0.88392 1.9812) (xy 0.77216 2.02692) (xy 0.68834 2.06502)
+      (xy 0.65024 2.08788) (xy 0.6477 2.09042) (xy 0.635 2.13868) (xy 0.61214 2.23774)
+      (xy 0.58166 2.3749) (xy 0.55118 2.54) (xy 0.5461 2.5654) (xy 0.51562 2.72542)
+      (xy 0.49022 2.85496) (xy 0.47244 2.9464) (xy 0.46228 2.9845) (xy 0.43942 2.98958)
+      (xy 0.36322 2.99466) (xy 0.24384 2.9972) (xy 0.1016 2.99974) (xy -0.0508 2.99974)
+      (xy -0.19812 2.99466) (xy -0.32258 2.99212) (xy -0.41402 2.9845) (xy -0.45212 2.97688)
+      (xy -0.45212 2.97434) (xy -0.46736 2.92608) (xy -0.48768 2.82702) (xy -0.51562 2.68732)
+      (xy -0.54864 2.52476) (xy -0.55372 2.49428) (xy -0.5842 2.3368) (xy -0.6096 2.20726)
+      (xy -0.62992 2.11582) (xy -0.64008 2.08026) (xy -0.65278 2.07264) (xy -0.71882 2.0447)
+      (xy -0.8255 2.00152) (xy -0.95758 1.94818) (xy -1.26238 1.82372) (xy -1.6383 2.08026)
+      (xy -1.67132 2.10312) (xy -1.80594 2.1971) (xy -1.9177 2.27076) (xy -1.9939 2.31902)
+      (xy -2.02692 2.3368) (xy -2.02946 2.3368) (xy -2.06756 2.30378) (xy -2.14122 2.2352)
+      (xy -2.24282 2.13614) (xy -2.35966 2.01676) (xy -2.44856 1.9304) (xy -2.55016 1.82626)
+      (xy -2.6162 1.75514) (xy -2.65176 1.70942) (xy -2.66446 1.68148) (xy -2.66192 1.6637)
+      (xy -2.63652 1.6256) (xy -2.58318 1.54178) (xy -2.50444 1.43002) (xy -2.413 1.2954)
+      (xy -2.33934 1.18618) (xy -2.25806 1.05918) (xy -2.20472 0.97028) (xy -2.18694 0.9271)
+      (xy -2.19202 0.90678) (xy -2.21742 0.83566) (xy -2.2606 0.7239) (xy -2.31902 0.59182)
+      (xy -2.44856 0.29464) (xy -2.6416 0.25654) (xy -2.76098 0.23622) (xy -2.92608 0.2032)
+      (xy -3.08356 0.17272) (xy -3.32994 0.12446) (xy -3.33756 -0.77978) (xy -3.29946 -0.79502)
+      (xy -3.2639 -0.80518) (xy -3.17246 -0.8255) (xy -3.04292 -0.8509) (xy -2.88798 -0.87884)
+      (xy -2.75844 -0.90424) (xy -2.62636 -0.92964) (xy -2.52984 -0.94742) (xy -2.4892 -0.95758)
+      (xy -2.47904 -0.97028) (xy -2.44602 -1.03378) (xy -2.39776 -1.13538) (xy -2.34696 -1.2573)
+      (xy -2.29362 -1.3843) (xy -2.2479 -1.50114) (xy -2.21488 -1.59004) (xy -2.20218 -1.6383)
+      (xy -2.21996 -1.67132) (xy -2.27076 -1.75006) (xy -2.34188 -1.85928) (xy -2.43332 -1.99136)
+      (xy -2.52222 -2.1209) (xy -2.59842 -2.2352) (xy -2.64922 -2.31394) (xy -2.67208 -2.35204)
+      (xy -2.66192 -2.37744) (xy -2.60858 -2.44094) (xy -2.50952 -2.54254) (xy -2.3622 -2.68732)
+      (xy -2.33934 -2.71018) (xy -2.2225 -2.82448) (xy -2.12344 -2.91592) (xy -2.05486 -2.97688)
+      (xy -2.02438 -2.99974)) (layer B.SilkS) (width 0.00254))
+  )
   (gr_text "BAT<          >USB" (at 121.793 101.6 90) (layer B.SilkS)
