File: kicad/feather_v3/feather_v3.kicad_pcb (KiCad board)
At the start: 2 copper layers, 52.1 x 52.1 mm, 12 parts, among them P1 Input1, P2 Output1, P3 5V, P4 GND, P5 Input2, P6 Output2, P7 CI_A, P9 DI_A

Commit message: clean up of all kicad project folders
Parts:
- added L1: LOGO_U88, feather_v3:logo_ultim8x8_small, F.Cu at (121.9, 106.7)
- added L2: OSHW, feather_v3:OSHW_6mm, F.Cu at (121.9, 123.8)
- L3: value WyoLum -> LOGO_WL
- L4: value Maniacal Labs -> LOGO_ML
- moved L3 3.59 mm to (114.3, 99.1)
- moved L4 2.54 mm to (114.3, 132.1)
