File: kicad/ultim_bus/ultim_bus.kicad_pcb (KiCad board)
At the start: 2 copper layers, 198.1 x 55.9 mm, 154 parts, among them M1 MouseBite, M10 MouseBite, M11 MouseBite, M12 MouseBite, M13 MouseBite, M14 MouseBite, M15 MouseBite, M16 MouseBite, M17 MouseBite, M18 MouseBite, M2 MouseBite, M3 MouseBite, M4 MouseBite, M5 MouseBite, M6 MouseBite, M7 MouseBite, M8 MouseBite, M9 MouseBite, P1 CONN_1, P10 CONN_1, P11 CONN_1, P12 CONN_1, P13 CONN_1, P14 CONN_1, P15 CONN_1, P16 CONN_1, P17 CONN_1, P18 CONN_1, P19 CONN_1, P2 CONN_1, P20 CONN_1, P21 CONN_1, P22 CONN_1, P23 CONN_1, P24 CONN_1, P25 CONN_1, P26 CONN_1, P27 CONN_1, P28 CONN_1, P29 CONN_1, P3 CONN_1, P30 CONN_1, P31 CONN_1, P32 CONN_1, P33 CONN_1, P34 CONN_1, P35 CONN_1, P36 CONN_1, P37 CONN_1, P38 CONN_1, P39 CONN_1, P4 CONN_1, P40 CONN_1, P41 CONN_1, P42 CONN_1, P43 CONN_1, P44 CONN_1, P45 CONN_1, P46 CONN_1, P47 CONN_1, P48 CONN_1, P49 CONN_1, P5 CONN_1, P50 CONN_1, P51 CONN_1, P52 CONN_1, P6 CONN_1, P7 CONN_1, P8 CONN_1, P9 CONN_1

Commit message: clean up of all kicad project folders
Parts:
- removed REF**111, REF**1111 (x2), REF**11111 (x3), REF**1111111 (x2), REF**11111110 (x2), REF**1111112 (x2), REF**1111113 (x2), REF**1111114 (x2), REF**1111115 (x2), REF**1111116 (x2), REF**1111117 (x2), REF**1111118 (x2), REF**11112 (x3), REF**11113 (x3), REF**11114 (x3), REF**11115 (x3), REF**11116 (x3), REF**11117 (x3), REF**11118 (x6), REF**1112 (x2), REF**1113 (x2), REF**1114 (x2), REF**1115 (x2), REF**1116 (x2), REF**1117 (x2), REF**1118 (x2), REF**1119 (x2), REF**112, REF**113, REF**114, REF**115, REF**116, REF**117, REF**118, REF**119: via_0.8, ultim8x8_libs:via_0.8
- added v1: via_0.8x9, ultim_bus:via_0.8x9, F.Cu at (210.8, 30.5)
- added v10: via_0.8x9, ultim_bus:via_0.8x9, F.Cu at (210.8, 61.0)
- added v11: via_0.8x9, ultim_bus:via_0.8x9, F.Cu at (149.9, 61.0)
- added v12: via_0.8x9, ultim_bus:via_0.8x9, F.Cu at (88.9, 61.0)
- added v2: via_0.8x9, ultim_bus:via_0.8x9, F.Cu at (149.9, 30.5)
- added v3: via_0.8x9, ultim_bus:via_0.8x9, F.Cu at (88.9, 30.5)
- added v4: via_0.8x9, ultim_bus:via_0.8x9, F.Cu at (210.8, 76.2)
- added v5: via_0.8x9, ultim_bus:via_0.8x9, F.Cu at (149.9, 76.2)
- added v6: via_0.8x9, ultim_bus:via_0.8x9, F.Cu at (88.9, 76.2)
- added v7: via_0.8x9, ultim_bus:via_0.8x9, F.Cu at (210.8, 45.7)
- added v8: via_0.8x9, ultim_bus:via_0.8x9, F.Cu at (149.9, 45.7)
- added v9: via_0.8x9, ultim_bus:via_0.8x9, F.Cu at (88.9, 45.7)
- L10, L3, L5, L8: moved to B.Cu
- moved L5 31.1 mm to (135.3, 61.0), turned to 180 degrees
- moved L3 30.5 mm to (134.6, 30.5), turned to 180 degrees
- moved L4 30.5 mm to (134.6, 45.7)
- moved L6 30.5 mm to (134.6, 76.2)
- turned L10 to 180 degrees
- turned L8 to 180 degrees
Connections:
- net /ROW1 renamed /5V
- net /ROW2 renamed /GND
- net /ROW31 renamed /CLK3
- net /ROW32 renamed /CLK2
- net /ROW33 renamed /CLK1
- net /ROW34 renamed /CLK
- net /ROW41 renamed /DAT3
- net /ROW42 renamed /DAT2
- net /ROW43 renamed /DAT1
- net /ROW44 renamed /DAT
Routing:
- net /GND: track 30.5 -> 7.62 mm
- net /5V: track 30.5 -> 7.62 mm
- net /DAT2: track 0.00 -> 2.54 mm
- net /DAT1: track 0.00 -> 2.54 mm
- net /CLK2: track 0.00 -> 2.54 mm
- net /CLK1: track 0.00 -> 2.54 mm
Other:
- board text added: "IN"
- board text added: "OUT"
