File: kicad/ultim_bus/ultim_bus.sch (KiCad schematic (older format))
At the start: 82 parts, among them M1 MouseBite, M10 MouseBite, M11 MouseBite, M12 MouseBite, M13 MouseBite, M14 MouseBite, M15 MouseBite, M16 MouseBite, M17 MouseBite, M18 MouseBite, M2 MouseBite, M3 MouseBite, M4 MouseBite, M5 MouseBite, M6 MouseBite, M7 MouseBite, M8 MouseBite, M9 MouseBite, P1 CONN_1, P10 CONN_1, P11 CONN_1, P12 CONN_1, P13 CONN_1, P14 CONN_1, P15 CONN_1, P16 CONN_1, P17 CONN_1, P18 CONN_1, P19 CONN_1, P2 CONN_1, P20 CONN_1, P21 CONN_1, P22 CONN_1, P23 CONN_1, P24 CONN_1, P25 CONN_1, P26 CONN_1, P27 CONN_1, P28 CONN_1, P29 CONN_1, P3 CONN_1, P30 CONN_1, P31 CONN_1, P32 CONN_1, P33 CONN_1, P34 CONN_1, P35 CONN_1, P36 CONN_1, P37 CONN_1, P38 CONN_1, P39 CONN_1, P4 CONN_1, P40 CONN_1, P41 CONN_1, P42 CONN_1, P43 CONN_1, P44 CONN_1, P45 CONN_1, P46 CONN_1, P47 CONN_1, P48 CONN_1, P49 CONN_1, P5 CONN_1, P50 CONN_1, P51 CONN_1, P52 CONN_1, P6 CONN_1, P7 CONN_1, P8 CONN_1, P9 CONN_1

Commit message: clean up of all kicad project folders
Parts:
- added v1, v10, v11, v12, v2, v3, v4, v5, v6, v7, v8, v9: via_0.8x9, ultim_bus:via_0.8x9, symbol via_0.8x9
- L1, L2: footprint ultim8x8_libs:OSHW_6mm -> ultim_bus:OSHW_6mm; symbol CONN_1 -> OSHW
- L10, L7, L8, L9: footprint ultim8x8_libs:logo_MLlabs_small -> ultim_bus:logo_MLlabs_small; symbol CONN_1 -> LOGO_ML
- L11, L12: footprint ultim8x8_libs:logo_ultim8x8_small -> ultim_bus:logo_ultim8x8_small; symbol CONN_1 -> LOGO_U88
- L3, L4, L5, L6: footprint ultim8x8_libs:logo_wyo_butterfly_small -> ultim_bus:logo_wyo_butterfly_small; symbol CONN_1 -> LOGO_WL
- M1, M10, M11, M15, M16, M17, M18, M2, M3, M4, M8, M9: footprint ultim8x8_libs:mouse-bite-5.08mm-slot -> ultim_bus:mouse-bite-5.08mm-slot
- M12, M13, M14, M5, M6, M7: footprint ultim8x8_libs:mouse-bite-2.54mm-slot -> ultim_bus:mouse-bite-2.54mm-slot
- P1, P12, P15, P16, P19, P20, P23, P24, P32, P33, P36, P37, P4, P40, P43, P44, P47, P48, P5, P51, P8, P9: footprint ultim8x8_libs:Screw_SqPad -> ultim_bus:Screw_SqPad
- P10, P11, P13, P14, P17, P18, P2, P21, P22, P25, P26, P27, P3, P30, P31, P34, P35, P38, P39, P41, P42, P45, P46, P49, P50, P52, P6, P7: footprint ultim8x8_libs:Screw -> ultim_bus:Screw
- P28, P29: footprint ultim8x8_libs:Screw_SqPad -> ultim_bus:Screw_SSide
Connections:
- net ROW1 renamed 5V
- net 5V: now also v1.1, v1.2, v1.3, v1.4, v1.5, v1.6, v1.7, v1.8, v1.9, v2.1, v2.2, v2.3, v2.4, v2.5, v2.6, v2.7, v2.8, v2.9, v3.1, v3.2, v3.3, v3.4, v3.5, v3.6, v3.7, v3.8, v3.9
- net ROW2 renamed GND
- net GND: now also v4.1, v4.2, v4.3, v4.4, v4.5, v4.6, v4.7, v4.8, v4.9, v5.1, v5.2, v5.3, v5.4, v5.5, v5.6, v5.7, v5.8, v5.9, v6.1, v6.2, v6.3, v6.4, v6.5, v6.6, v6.7, v6.8, v6.9
- net ROW31 renamed CLK3
- net ROW32 renamed CLK2
- net CLK2: now also v9.1, v9.2, v9.3, v9.4, v9.5, v9.6, v9.7, v9.8, v9.9
- net ROW33 renamed CLK1
- net CLK1: now also v8.1, v8.2, v8.3, v8.4, v8.5, v8.6, v8.7, v8.8, v8.9
- net ROW34 renamed CLK
- net CLK: now also v7.1, v7.2, v7.3, v7.4, v7.5, v7.6, v7.7, v7.8, v7.9
- net ROW41 renamed DAT3
- net ROW42 renamed DAT2
- net DAT2: now also v12.1, v12.2, v12.3, v12.4, v12.5, v12.6, v12.7, v12.8, v12.9
- net ROW43 renamed DAT1
- net DAT1: now also v11.1, v11.2, v11.3, v11.4, v11.5, v11.6, v11.7, v11.8, v11.9
- net ROW44 renamed DAT
- net DAT: now also v10.1, v10.2, v10.3, v10.4, v10.5, v10.6, v10.7, v10.8, v10.9
- no-connect marks 30 -> 18
Other:
- note added: "LOGOS"
- moved on the sheet: M1, M10, M11, M12, M13, M14, M15, M16, M17, M18, M2, M3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
