File: kicad/ultim_bus_v3/ultim_bus.sch (KiCad schematic (older format))
At the start: 97 parts, among them M10 MouseBite, M11 MouseBite, M13 MouseBite, M16 MouseBite, M17 MouseBite, M18 MouseBite, M2 MouseBite, M3 MouseBite, M4 MouseBite, M6 MouseBite, M9 MouseBite, P1 CONN_1, P10 CONN_1, P11 CONN_1, P12 CONN_1, P14 CONN_1, P15 CONN_1, P16 CONN_1, P17 CONN_1, P18 CONN_1, P19 CONN_1, P2 CONN_1, P20 CONN_1, P21 CONN_1, P22 CONN_1, P23 CONN_1, P24 CONN_1, P25 CONN_1, P27 CONN_1, P28 CONN_1, P29 CONN_1, P3 CONN_1, P30 CONN_1, P31 CONN_1, P32 CONN_1, P33 CONN_1, P34 CONN_1, P35 CONN_1, P36 CONN_1, P37 CONN_1, P38 CONN_1, P4 CONN_1, P40 CONN_1, P41 CONN_1, P42 CONN_1, P43 CONN_1, P44 CONN_1, P45 CONN_1, P46 CONN_1, P47 CONN_1, P48 CONN_1, P49 CONN_1, P5 CONN_1, P50 CONN_1, P51 CONN_1, P6 CONN_1, P7 CONN_1, P8 CONN_1, P9 CONN_1

Commit message: Bus Bar PCB added El. Cap, removed short to GND
Parts:
- added C1: 470uF 10V, ultim_bus:cap_pol_rad3, symbol C_POL_1
- M10, M11, M13, M16, M17, M18, M2, M3, M4, M6, M9: symbol CONN_1 -> Mouse_Bite
Connections:
- net 5V: now also C1.1 (+)
- net GND: now also C1.2 (-); no longer H1.28 (GND)
- no-connect marks 27 -> 17
Other:
- note added: "Capacitors, Electrolytic, for filtering"
- note added: "Vias, for the snap-offs"
- moved on the sheet: H1, JP1, R1, R2, R3, R4, R5, R6, S1, S2, S3, S4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
