File: kicad/ultim_bus_v4/ultim_bus.sch (KiCad schematic (older format))
At the start: 98 parts, among them M10 MouseBite, M11 MouseBite, M13 MouseBite, M16 MouseBite, M17 MouseBite, M18 MouseBite, M2 MouseBite, M3 MouseBite, M4 MouseBite, M6 MouseBite, M9 MouseBite, P1 CONN_1, P10 CONN_1, P11 CONN_1, P12 CONN_1, P14 CONN_1, P15 CONN_1, P16 CONN_1, P17 CONN_1, P18 CONN_1, P19 CONN_1, P2 CONN_1, P20 CONN_1, P21 CONN_1, P22 CONN_1, P23 CONN_1, P24 CONN_1, P25 CONN_1, P27 CONN_1, P28 CONN_1, P29 CONN_1, P3 CONN_1, P30 CONN_1, P31 CONN_1, P32 CONN_1, P33 CONN_1, P34 CONN_1, P35 CONN_1, P36 CONN_1, P37 CONN_1, P38 CONN_1, P4 CONN_1, P40 CONN_1, P41 CONN_1, P42 CONN_1, P43 CONN_1, P44 CONN_1, P45 CONN_1, P46 CONN_1, P47 CONN_1, P48 CONN_1, P49 CONN_1, P5 CONN_1, P50 CONN_1, P51 CONN_1, P6 CONN_1, P7 CONN_1, P8 CONN_1, P9 CONN_1

Commit message: add feather huzzah footprint
Parts:
- H1: symbol FeatherM0 -> FeatherHuzzah
Connections:
- net A0: no longer H1.17 (A0)
- net A1: no longer names the net of R2.1, S2.1
- net A1: no longer H1.18 (A1)
- net A2: no longer names the net of R3.1, S3.1
- net A2: no longer H1.19 (A2)
- net A3: no longer names the net of R4.1, S4.1
- net A3: no longer H1.20 (A3)
- net A4: no longer names the net of R5.1, S5.1
- net A4: no longer H1.21 (A4)
- net A5: no longer names the net of R6.1, S6.1
- net A5: no longer H1.22 (A5)
- no-connect marks 17 -> 19
Changed lines of the file:
@@
 NoConn ~ 7775 2075
 NoConn ~ 7775 1975
-NoConn ~ 7775 1875
-NoConn ~ 7775 1775
-NoConn ~ 7775 1675
-NoConn ~ 7775 1575
 NoConn ~ 7775 1375
 $Comp
@@
 	10950 1800 10950 900
 $Comp
-L FeatherM0 H1
+L FeatherHuzzah H1
 U 1 1 58E305D1
 P 6675 2375
@@
 Wire Wire Line
 	6475 1275 6100 1275
-Text Label 6100 1275 0    50   ~ 10
-A0
-Text Label 6100 1375 0    50   ~ 10
-A1
-Text Label 6100 1475 0    50   ~ 10
-A2
-Text Label 6100 1575 0    50   ~ 10
-A3
-Text Label 6100 1675 0    50   ~ 10
-A4
-Text Label 6100 1775 0    50   ~ 10
-A5
 Wire Wire Line
 	9300 2250 9300 2100
@@
 Text Label 8700 2100 0    50   ~ 10
 A0
-Text Label 8700 2375 0    50   ~ 10
-A1
-Text Label 8700 2625 0    50   ~ 10
-A2
-Text Label 8700 2875 0    50   ~ 10
-A3
-Text Label 8700 3125 0    50   ~ 10
-A4
-Text Label 8700 3375 0    50   ~ 10
-A5
 Wire Notes Line
 	8450 2000 10950 2000
@@
 Wire Wire Line
 	8550 4575 8800 4575
+NoConn ~ 6100 1275
+NoConn ~ 6100 1375
+NoConn ~ 6100 1475
+NoConn ~ 6100 1575
+NoConn ~ 6100 1675
+NoConn ~ 6100 1775
 $EndSCHEMATC
