File: kicad/ultim_bus_v5/ultim_bus.kicad_pcb (KiCad board)
At the start: 2 copper layers, 177.8 x 55.9 mm, 98 parts, among them M10 MouseBite, M11 MouseBite, M13 MouseBite, M16 MouseBite, M17 MouseBite, M18 MouseBite, M2 MouseBite, M3 MouseBite, M4 MouseBite, M6 MouseBite, M9 MouseBite, P1 CONN_1, P10 CONN_1, P11 CONN_1, P12 CONN_1, P14 CONN_1, P15 CONN_1, P16 CONN_1, P17 CONN_1, P18 CONN_1, P19 CONN_1, P2 CONN_1, P20 CONN_1, P21 CONN_1, P22 CONN_1, P23 CONN_1, P24 CONN_1, P25 CONN_1, P27 CONN_1, P28 CONN_1, P29 CONN_1, P3 CONN_1, P30 CONN_1, P31 CONN_1, P32 CONN_1, P33 CONN_1, P34 CONN_1, P35 CONN_1, P36 CONN_1, P37 CONN_1, P38 CONN_1, P4 CONN_1, P40 CONN_1, P41 CONN_1, P42 CONN_1, P43 CONN_1, P44 CONN_1, P45 CONN_1, P46 CONN_1, P47 CONN_1, P48 CONN_1, P49 CONN_1, P5 CONN_1, P50 CONN_1, P51 CONN_1, P6 CONN_1, P7 CONN_1, P8 CONN_1, P9 CONN_1

Commit message: ultim_bus_v5 swappes S1 and S2
Parts:
- moved S1 11.4 mm to (126.4, 38.1)
- moved S2 11.4 mm to (137.8, 38.1)
Routing:
- net /S2: track 65.8 -> 52.9 mm
- net /S1: track 54.1 -> 64.8 mm
Changed lines of the file:
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@@
     (links 231)
     (no_connects 0)
-    (area 15.437055 18.89 224.055715 94.14)
+    (area 27.864999 25.324999 205.815001 81.355001)
     (thickness 1.6)
     (drawings 440)
-    (tracks 300)
+    (tracks 301)
     (zones 0)
     (modules 98)
@@
     (aux_axis_origin 27.94 81.28)
     (grid_origin 27.94 81.28)
-    (visible_elements FFFFFF7F)
+    (visible_elements FFFFEF7F)
     (pcbplotparams
-      (layerselection 0x010f0_80000001)
-      (usegerberextensions true)
-      (usegerberattributes true)
-      (excludeedgelayer true)
+      (layerselection 0x00130_80000001)
+      (usegerberextensions false)
+      (excludeedgelayer false)
       (linewidth 0.101600)
-      (plotframeref false)
+      (plotframeref true)
       (viasonmask false)
       (mode 1)
@@
       (plotvalue true)
       (plotinvisibletext false)
-      (padsonsilk false)
-      (subtractmaskfromsilk true)
-      (outputformat 1)
+      (padsonsilk true)
+      (subtractmaskfromsilk false)
+      (outputformat 4)
       (mirror false)
-      (drillshape 0)
+      (drillshape 2)
       (scaleselection 1)
-      (outputdirectory ultim_bus_gerber/))
+      (outputdirectory ultim_bus_pdf/))
   )
   (net 0 "")
@@
   )
   (module ultim_bus:SW-PB (layer F.Cu)
-    (at 137.795 38.1 90)
+    (at 126.365 38.1 90)
     (descr "PCB pushbutton, Tyco FSM6x6 series")
     (tags pushbutton)
@@
   )
   (module ultim_bus:SW-PB (layer F.Cu)
-    (at 126.365 38.1 90)
+    (at 137.795 38.1 90)
     (descr "PCB pushbutton, Tyco FSM6x6 series")
     (tags pushbutton)
@@
     (effects (font (size 1.27 1.27) (thickness 0.254)) (justify mirror))
   )
-  (gr_text S2 (at 126.365 38.1) (layer B.SilkS)
+  (gr_text S1 (at 126.365 38.1) (layer B.SilkS)
     (effects (font (size 1.27 1.27) (thickness 0.254)) (justify mirror))
   )
-  (gr_text S1 (at 137.795 38.1) (layer B.SilkS)
+  (gr_text S2 (at 137.795 38.1) (layer B.SilkS)
     (effects (font (size 1.27 1.27) (thickness 0.254)) (justify mirror))
   )
@@
   (segment (start 149.606 41.402) (end 149.606 53.34) (width 0.25) (layer B.Cu) (net 14))
   (segment (start 129.615 55.59) (end 123.115 55.59) (width 0.25) (layer F.Cu) (net 14) (status 30))
+  (segment (start 143.002 42.799) (end 143.383 43.18) (width 0.25) (layer F.Cu) (net 15))
+  (segment (start 141.045 40.35) (end 142.302235 40.35) (width 0.25) (layer F.Cu) (net 15))
+  (segment (start 142.302235 40.35) (end 143.002 41.049765) (width 0.25) (layer F.Cu) (net 15))
+  (segment (start 143.002 41.049765) (end 143.002 42.799) (width 0.25) (layer F.Cu) (net 15))
+  (segment (start 134.545 40.35) (end 141.045 40.35) (width 0.25) (layer F.Cu) (net 15))
   (segment (start 151.638 40.767) (end 150.749 40.767) (width 0.25) (layer B.Cu) (net 15))
   (segment (start 154.649 40.767) (end 157.255 38.161) (width 0.25) (layer B.Cu) (net 15))
@@
   (segment (start 149.943736 43.18) (end 150.368 43.18) (width 0.25) (layer F.Cu) (net 15))
   (segment (start 143.383 43.18) (end 149.943736 43.18) (width 0.25) (layer F.Cu) (net 15))
-  (segment (start 142.367 39.751) (end 142.367 42.164) (width 0.25) (layer F.Cu) (net 15))
-  (segment (start 129.615 40.35) (end 130.976 38.989) (width 0.25) (layer F.Cu) (net 15))
-  (segment (start 141.605 38.989) (end 142.367 39.751) (width 0.25) (layer F.Cu) (net 15))
-  (segment (start 142.367 42.164) (end 143.383 43.18) (width 0.25) (layer F.Cu) (net 15))
   (via (at 150.368 43.18) (size 0.6) (drill 0.4) (layers F.Cu B.Cu) (net 15))
-  (segment (start 130.976 38.989) (end 141.605 38.989) (width 0.25) (layer F.Cu) (net 15))
-  (segment (start 123.115 40.35) (end 129.615 40.35) (width 0.25) (layer F.Cu) (net 15) (status 30))
+  (segment (start 133.731 41.783) (end 141.220765 41.783) (width 0.25) (layer F.Cu) (net 16))
+  (segment (start 141.220765 41.783) (end 143.51 44.072235) (width 0.25) (layer F.Cu) (net 16))
+  (segment (start 132.298 40.35) (end 133.731 41.783) (width 0.25) (layer F.Cu) (net 16))
+  (segment (start 129.615 40.35) (end 132.298 40.35) (width 0.25) (layer F.Cu) (net 16))
+  (segment (start 123.115 40.35) (end 129.615 40.35) (width 0.25) (layer F.Cu) (net 16))
   (segment (start 152.654 41.275) (end 151.510992 41.275) (width 0.25) (layer B.Cu) (net 16))
   (segment (start 152.654 41.275) (end 156.3 41.275) (width 0.25) (layer B.Cu) (net 16))
@@
   (segment (start 152.018992 52.07) (end 151.129992 51.181) (width 0.25) (layer B.Cu) (net 16))
   (segment (start 151.129992 46.144264) (end 151.129992 45.72) (width 0.25) (layer B.Cu) (net 16))
-  (segment (start 141.045 40.35) (end 141.045 41.607235) (width 0.25) (layer F.Cu) (net 16))
   (segment (start 143.51 45.339) (end 143.891 45.72) (width 0.25) (layer F.Cu) (net 16))
   (segment (start 143.51 44.072235) (end 143.51 45.339) (width 0.25) (layer F.Cu) (net 16))
@@
   (segment (start 150.705728 45.72) (end 151.129992 45.72) (width 0.25) (layer F.Cu) (net 16))
   (segment (start 143.891 45.72) (end 150.705728 45.72) (width 0.25) (layer F.Cu) (net 16))
-  (segment (start 141.045 41.607235) (end 143.51 44.072235) (width 0.25) (layer F.Cu) (net 16))
-  (segment (start 141.045 40.35) (end 134.545 40.35) (width 0.25) (layer F.Cu) (net 16) (status 30))
   (zone (net 1) (net_name /GND) (layer F.Cu) (hatch edge 0.508)
     (connect_pads (clearance 0.508))
