File: kicad/ultim_8x8_v2/ultim8x8.sch (KiCad schematic (older format))
At the start: 24 parts, among them P1 Input1, P10 DO_H, P11 5V, P12 GND, P13 CI_A, P14 CO_H, P15 DI_A, P16 DO_H, P17 5V, P18 5V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

Commit message: U88 ver2 with extra power / signal mounting holes
Parts:
- L1: footprint ultim8x8_libs:logo_ultim8x8 -> ultim8x8_libs:logo_ultim8x8_7mm
- L3: footprint ultim8x8_libs:logo_wyo_butterfly -> ultim8x8_libs:logo_wyo_butterfly_5mm
- L4: footprint ultim8x8_libs:logo_MLlabs -> ultim8x8_libs:logo_MLlabs_5mm
Changed lines of the file:
@@
 F 0 "L3" H 10525 6100 40  0000 C CNN
 F 1 "Wyolum" H 10425 6250 30  0001 C CNN
-F 2 "ultim8x8_libs:logo_wyo_butterfly" H 10450 6325 30  0001 C CNN
+F 2 "ultim8x8_libs:logo_wyo_butterfly_5mm" H 10450 6325 30  0001 C CNN
 F 3 "" H 10525 6250 60  0001 C CNN
 F 4 "mfr_pn" H 10525 6250 60  0001 C CNN "manf#"
@@
 F 0 "L4" H 10875 5875 40  0000 C CNN
 F 1 "Maniacal Labs" H 10775 6125 30  0001 C CNN
-F 2 "ultim8x8_libs:logo_MLlabs" H 10800 6200 30  0001 C CNN
+F 2 "ultim8x8_libs:logo_MLlabs_5mm" H 10800 6200 30  0001 C CNN
 F 3 "" H 10875 6125 60  0001 C CNN
 F 4 "mfr_pn" H 10875 6125 60  0001 C CNN "manf#"
@@
 F 0 "L1" H 9325 5850 40  0000 C CNN
 F 1 "ULTiM8x8" H 9225 6125 30  0001 C CNN
-F 2 "ultim8x8_libs:logo_ultim8x8" H 9325 6280 30  0001 C CNN
+F 2 "ultim8x8_libs:logo_ultim8x8_7mm" H 9325 6280 30  0001 C CNN
 F 3 "" H 9325 6125 60  0001 C CNN
 F 4 "mfr_pn" H 9325 6125 60  0001 C CNN "manf#"
